File: hw/audio-1/audio-1.kicad_pcb (KiCad board)
At the start: 2 copper layers, 108.5 x 47 mm, 75 parts, among them J1 Conn_01x03, J2 Conn_01x04, J3 Conn_01x04, J4 Conn_01x04, U1 LM4562, U2 LM4562, U3 LM4562, U4 LM4562, U5 SN74LVC1G3157DBVR, U6 SN74LVC1G3157DBVR

Commit message: Version used to generage gerbers
Parts:
- J1: value Conn_01x03 -> Conn_01x02; footprint Connector_PinHeader_2.54mm:PinHeader_1x03_P2.54mm_Vertical -> Connector_PinHeader_2.54mm:PinHeader_1x02_P2.54mm_Vertical
- moved J1 5.74 mm to (163.0, 81.5), turned to 0 degrees
Connections:
- J1 pad 2: +3.3V -> GND
Routing:
- net +5V: track 153.2 -> 147.0 mm
- net Net-(C14-Pad2): track 25.8 -> 28.1 mm
Other:
- board text removed: "3.3"

Commit message: Version used to generage gerbers
Parts:
- moved H1 0.50 mm to (140.0, 51.0)
Changed lines of the file:
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@@
 			(plot_on_all_layers_selection 0x0000000_00000000)
 			(disableapertmacros no)
-			(usegerberextensions no)
-			(usegerberattributes yes)
-			(usegerberadvancedattributes yes)
-			(creategerberjobfile yes)
+			(usegerberextensions yes)
+			(usegerberattributes no)
+			(usegerberadvancedattributes no)
+			(creategerberjobfile no)
 			(dashed_line_dash_ratio 12.000000)
 			(dashed_line_gap_ratio 3.000000)
@@
 			(psa4output no)
 			(plotreference yes)
-			(plotvalue yes)
+			(plotvalue no)
 			(plotfptext yes)
 			(plotinvisibletext no)
 			(sketchpadsonfab no)
-			(subtractmaskfromsilk no)
+			(subtractmaskfromsilk yes)
 			(outputformat 1)
 			(mirror no)
-			(drillshape 1)
+			(drillshape 0)
 			(scaleselection 1)
-			(outputdirectory "")
+			(outputdirectory "plots/")
 		)
 	)
@@
 	(footprint "MountingHole:MountingHole_3.5mm"
 		(layer "F.Cu")
-		(at 140 50.5)
+		(at 140 51)
 		(descr "Mounting Hole 3.5mm, no annular")
 		(tags "mounting hole 3.5mm no annular")
