File: hw/audio-1/audio-in.kicad_sch (KiCad schematic)
At the start: 24 parts, among them U1 LM4562, U2 LM4562

Commit message: Version used to generage gerbers
Other:
- company: (none) -> KC1FSZ
- title: (none) -> Simple Repeater Controller
Changed lines of the file:
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@@
 	(generator "eeschema")
 	(generator_version "8.0")
-	(paper "A4")
+	(paper "USLetter")
+	(title_block
+		(title "Simple Repeater Controller")
+		(date "2025-01-16")
+		(rev "1")
+		(company "KC1FSZ")
+		(comment 1 "Copyright (C) 2025")
+		(comment 2 "For Non-Commercial Use Only")
+	)
 	(junction
 		(at 171.45 71.12)
