File: hw/audio-1/audio-mux.kicad_sch (KiCad schematic)
At the start: 2 parts, among them U5 SN74LVC1G3157DBVR, U6 SN74LVC1G3157DBVR

Commit message: Version used to generage gerbers
Other:
- company: (none) -> KC1FSZ
- title: (none) -> Simple Repeater Controller
Changed lines of the file:
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@@
 	(generator "eeschema")
 	(generator_version "8.0")
-	(paper "A4")
+	(paper "USLetter")
+	(title_block
+		(title "Simple Repeater Controller")
+		(date "2025-01-16")
+		(rev "1")
+		(company "KC1FSZ")
+		(comment 1 "Copyright (C) 2025")
+		(comment 2 "For Non-Commercial Use Only")
+	)
 	(junction
 		(at 113.03 63.5)
