File: hw/audio-1/audio-out.kicad_sch (KiCad schematic)
At the start: 37 parts, among them U3 LM4562, U4 LM4562

Commit message: Version used to generage gerbers
Other:
- company: (none) -> KC1FSZ
- title: (none) -> Simple Repeater Controller
Changed lines of the file:
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@@
 	(generator "eeschema")
 	(generator_version "8.0")
-	(paper "A4")
+	(paper "USLetter")
+	(title_block
+		(title "Simple Repeater Controller")
+		(date "2025-01-16")
+		(rev "1")
+		(company "KC1FSZ")
+		(comment 1 "Copyright (C) 2025")
+		(comment 2 "For Non-Commercial Use Only")
+	)
 	(junction
 		(at 238.76 74.93)

Commit message: Docs improvements
Parts:
- C12, C22: value C_Small -> 0.001uF
Changed lines of the file:
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@@
 			)
 		)
-		(property "Value" "C_Small"
+		(property "Value" "0.001uF"
 			(at 241.3 149.8662 0)
 			(effects
@@
 		(on_board yes)
 		(dnp no)
-		(fields_autoplaced yes)
 		(property "Reference" "#FLG07"
 			(at 152.4 36.195 0)
@@
 		)
 		(property "Value" "PWR_FLAG"
-			(at 152.4 33.02 0)
+			(at 159.766 32.004 0)
 			(effects
 				(font
@@
 		(on_board yes)
 		(dnp no)
-		(fields_autoplaced yes)
 		(property "Reference" "#FLG08"
 			(at 152.4 104.775 0)
@@
 		)
 		(property "Value" "PWR_FLAG"
-			(at 152.4 101.6 0)
+			(at 156.972 101.854 0)
 			(effects
 				(font
@@
 			)
 		)
-		(property "Value" "C_Small"
+		(property "Value" "0.001uF"
 			(at 241.3 81.2862 0)
 			(effects

Commit message: Working on 2
Parts:
- removed C14, C15, C18, C19, C20: 1uF, Capacitor_SMD:C_0805_2012Metric_Pad1.18x1.45mm_HandSolder, symbol Device:C_Small
- removed C17: 100pF, Capacitor_SMD:C_0805_2012Metric_Pad1.18x1.45mm_HandSolder, symbol Device:C_Small
- removed C21: 10uF, Capacitor_SMD:C_0805_2012Metric_Pad1.18x1.45mm_HandSolder, symbol Device:C_Small
- removed C22: 0.001uF, Capacitor_SMD:C_0805_2012Metric_Pad1.18x1.45mm_HandSolder, symbol Device:C_Small
- removed R14, R21, R22, R23, R25: 100k, Resistor_SMD:R_0805_2012Metric_Pad1.20x1.40mm_HandSolder, symbol Device:R_Small_US
- removed R24: 47, Resistor_SMD:R_0805_2012Metric_Pad1.20x1.40mm_HandSolder, symbol Device:R_Small_US
- removed R26: 200k, Resistor_SMD:R_0805_2012Metric_Pad1.20x1.40mm_HandSolder, symbol Device:R_Small_US
- removed R27, R28: 10k, Resistor_SMD:R_0805_2012Metric_Pad1.20x1.40mm_HandSolder, symbol Device:R_Small_US
- removed RV4: 50k, bruce-footprints:POT_3362P, symbol Device:R_Potentiometer_US
- removed TP4: TestPoint, TestPoint:TestPoint_Pad_3.0x3.0mm, symbol Connector:TestPoint
- removed U4: LM4562, Package_SO:SOIC-8_3.9x4.9mm_P1.27mm, symbol Amplifier_Operational:LM4562
