File: hw/control-1/control-1.kicad_sch (KiCad schematic)
At the start: 0 parts

Commit message: Control-1 sent to JLCPCB
Parts:
- added H1, H2, H3, H4: MountingHole, MountingHole:MountingHole_3.5mm, symbol Mechanical:MountingHole
- added J1: Conn_01x08, Connector_PinHeader_2.54mm:PinHeader_1x08_P2.54mm_Vertical, symbol Connector_Generic:Conn_01x08
- added J2: Conn_01x06, Connector_PinHeader_2.54mm:PinHeader_1x06_P2.54mm_Vertical, symbol Connector_Generic:Conn_01x06
Connections:
- new net +3.3V: J2.1 (Pin_1)
- new net COS0: J2.2 (Pin_2)
- new net COS1: J2.3 (Pin_3)
- new net GND: J2.6 (Pin_6)
- new net PTT0: J2.4 (Pin_4)
- new net PTT1: J2.5 (Pin_5)
- new net RADIO0-COS-N: J1.1 (Pin_1)
- new net RADIO0-COS-P: J1.2 (Pin_2)
- new net RADIO0-PTT-N: J1.6 (Pin_6)
- new net RADIO0-PTT-P: J1.5 (Pin_5)
- new net RADIO1-COS-N: J1.3 (Pin_3)
- new net RADIO1-COS-P: J1.4 (Pin_4)
- new net RADIO1-PTT-N: J1.8 (Pin_8)
- new net RADIO1-PTT-P: J1.7 (Pin_7)
Other:
- added sheet Power (power.kicad_sch)

Commit message: Working
Other:
- removed sheet Power
- company: (none) -> Bruce MacKinnon KC1FSZ
- title: (none) -> KC1FSZ Repeater Controller 1 - Radio Control Module
Changed lines of the file:
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@@
 	(generator "eeschema")
 	(generator_version "8.0")
-	(paper "A4")
+	(paper "USLetter")
+	(title_block
+		(title "KC1FSZ Repeater Controller 1 - Radio Control Module")
+		(date "2025-01-31")
+		(rev "1")
+		(company "Bruce MacKinnon KC1FSZ")
+		(comment 1 "Copyright (C) 2025 - Not for Commercial Use")
+	)
 	(junction
 		(at 161.29 96.52)
@@
 				)
 			)
-		)
-	)
-	(sheet
-		(at 73.66 27.94)
-		(size 36.83 34.29)
-		(fields_autoplaced yes)
-		(stroke
-			(width 0.1524)
-			(type solid)
-		)
-		(fill
-			(color 0 0 0 0.0000)
-		)
-		(property "Sheetname" "Power"
-			(at 73.66 27.2284 0)
-			(effects
-				(font
-					(size 1.27 1.27)
-				)
-				(justify left bottom)
-			)
-		)
-		(property "Sheetfile" "power.kicad_sch"
-			(at 73.66 62.8146 0)
-			(effects
-				(font
-					(size 1.27 1.27)
-				)
-				(justify left top)
-			)
-		)
-		(instances
-			(project "control-1"
-				(path "/010184a1-282b-4bd9-996b-54cd40db27a7"
-					(page "3")
-				)
-			)
