File: hw/control-1/radio-control.kicad_sch (KiCad schematic)
At the start: 10 parts, among them U1 LTV-356T, U2 LTV-356T, U3 LTV-356T, U4 LTV-356T

Commit message: Control-1 sent to JLCPCB
Connections:
- net GNDA renamed GND
- net RADIO0-PTT-A renamed RADIO0-PTT-P
- net RADIO0-PTT-B renamed RADIO0-PTT-N
- net RADIO1-PTT-A renamed RADIO1-PTT-P
- net RADIO1-PTT-B renamed RADIO1-PTT-N

Commit message: Working
Other:
- company: (none) -> Bruce MacKinnon KC1FSZ
- title: (none) -> KC1FSZ Repeater Controller 1 - Radio Control Module
Changed lines of the file:
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@@
 	(generator "eeschema")
 	(generator_version "8.0")
-	(paper "A4")
+	(paper "USLetter")
+	(title_block
+		(title "KC1FSZ Repeater Controller 1 - Radio Control Module")
+		(date "2025-01-31")
+		(rev "1")
+		(company "Bruce MacKinnon KC1FSZ")
+		(comment 1 "Copyright (C) 2025 - Not for Commercial Use")
+	)
 	(junction
 		(at 92.71 101.6)
