File: hw/if-2/controls.kicad_sch (KiCad schematic)
At the start: 0 parts

Commit message: Working on V2
Parts:
- added R22, R23, R24, R25, R32, R33, R34, R35: 1k, Resistor_SMD:R_0805_2012Metric_Pad1.20x1.40mm_HandSolder, symbol Device:R_US
- added R26, R27: 200, Resistor_SMD:R_0805_2012Metric_Pad1.20x1.40mm_HandSolder, symbol Device:R_US
- added U12, U13, U6, U7, U8, U9: LTV-356T, Package_SO:SO-4_4.4x3.6mm_P2.54mm, symbol Isolator:LTV-356T
Connections:
- new net: R33.2, U13.1
- new net: R26.2, U8.1
- new net: R22.2, U6.1
- new net: R32.2, U12.1
- new net: R27.2, U9.1
- new net: R23.2, U7.1
- new net +3.3V: R24.1, R25.1, R34.1, R35.1
- new net GND: U12.2, U12.3, U13.2, U13.3, U6.2, U6.3, U7.2, U7.3, U8.2, U8.3, U9.2, U9.3
- new net R0_COS: R22.1
- new net R0_COS_B: R24.2, U6.4
- new net R0_CTCSS: R32.1
- new net R0_CTCSS_B: R34.2, U12.4
- new net R0_PTT: U8.4
- new net R0_PTT_B: R26.1
- new net R1_COS: R23.1
- new net R1_COS_B: R25.2, U7.4
- new net R1_CTCSS: R33.1
- new net R1_CTCSS_B: R35.2, U13.4
- new net R1_PTT: U9.4
- new net R1_PTT_B: R27.1
Other:
- note added: "Converts 3.3V logic to pull PTT to ground."
- note added: "Converts radio COS signals to 3.3V logic."
- note added: "Converts radio CTCSS signals to 3.3V logic."
- note added: "TODO: Validate max current on LTV-353T input."
- title: Digital Repeater Controller  -> COS/PTT Controls

Commit message: First draft of schematic
Other:
- title: COS/PTT Controls -> COS/CTCSS/PTT Controls
Changed lines of the file:
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@@
 	(paper "USLetter")
 	(title_block
-		(title "COS/PTT Controls")
+		(title "COS/CTCSS/PTT Controls")
 		(date "2025-03-16")
 		(rev "2")
