File: hw/if-2/adc.kicad_sch (KiCad schematic)
At the start: 18 parts, among them U3 PCM1804DBR

Commit message: Working on 2
Other:
- title: Digital Repeater Controller  -> Analog To Digital Converter
Changed lines of the file:
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@@
 	(paper "USLetter")
 	(title_block
-		(title "Digital Repeater Controller ")
+		(title "Analog To Digital Converter")
 		(date "2025-03-16")
 		(rev "2")
@@
 	)
 	(junction
-		(at 171.45 93.98)
+		(at 167.64 93.98)
 		(diameter 0)
 		(color 0 0 0 0)
@@
 	)
 	(junction
-		(at 115.57 111.76)
+		(at 121.92 111.76)
 		(diameter 0)
 		(color 0 0 0 0)
@@
 	(wire
 		(pts
-			(xy 124.46 83.82) (xy 115.57 83.82)
+			(xy 124.46 83.82) (xy 121.92 83.82)
 		)
 		(stroke
@@
 	(wire
 		(pts
-			(xy 162.56 91.44) (xy 172.72 91.44)
+			(xy 162.56 91.44) (xy 170.18 91.44)
 		)
 		(stroke
@@
 	(wire
 		(pts
-			(xy 162.56 83.82) (xy 171.45 83.82)
+			(xy 162.56 83.82) (xy 167.64 83.82)
 		)
 		(stroke
@@
 	(wire
 		(pts
-			(xy 115.57 111.76) (xy 115.57 121.92)
+			(xy 121.92 111.76) (xy 121.92 121.92)
 		)
 		(stroke
@@
 	(wire
 		(pts
-			(xy 171.45 93.98) (xy 171.45 118.11)
+			(xy 167.64 93.98) (xy 167.64 120.65)
 		)
 		(stroke
@@
 	(wire
 		(pts
-			(xy 115.57 83.82) (xy 115.57 111.76)
-		)
-		(stroke
-			(width 0)
-			(type default)
-		)
-	)
-	(wire
-		(pts
-			(xy 171.45 83.82) (xy 171.45 93.98)
+			(xy 121.92 83.82) (xy 121.92 111.76)
+		)
+		(stroke
+			(width 0)
+			(type default)
+		)
+	)
+	(wire
+		(pts
+			(xy 167.64 83.82) (xy 167.64 93.98)
 		)
 		(stroke
@@
 	(wire
 		(pts
-			(xy 162.56 93.98) (xy 171.45 93.98)
+			(xy 162.56 93.98) (xy 167.64 93.98)
 		)
 		(stroke
@@
 	(wire
 		(pts
-			(xy 162.56 88.9) (xy 185.42 88.9)
-		)
-		(stroke
-			(width 0)
-			(type default)
-		)
-	)
-	(wire
-		(pts
-			(xy 115.57 111.76) (xy 124.46 111.76)
+			(xy 162.56 88.9) (xy 182.88 88.9)
+		)
+		(stroke
+			(width 0)
+			(type default)
+		)
+	)
+	(wire
+		(pts
+			(xy 121.92 111.76) (xy 124.46 111.76)
 		)
 		(stroke
@@
 	(global_label "R1_VIN-"
 		(shape input)
-		(at 172.72 91.44 0)
+		(at 170.18 91.44 0)
 		(fields_autoplaced yes)
 		(effects
@@
 		)
 		(property "Intersheetrefs" "${INTERSHEET_REFS}"
-			(at 183.7486 91.44 0)
+			(at 181.2086 91.44 0)
 			(effects
 				(font
@@
 	(global_label "R1_VIN+"
 		(shape input)
-		(at 185.42 88.9 0)
+		(at 182.88 88.9 0)
 		(fields_autoplaced yes)
 		(effects
@@
 		)
 		(property "Intersheetrefs" "${INTERSHEET_REFS}"
-			(at 196.4486 88.9 0)
+			(at 193.9086 88.9 0)
 			(effects
 				(font
@@
 	(symbol
 		(lib_id "power:GND")
-		(at 115.57 121.92 0)
+		(at 121.92 121.92 0)
 		(unit 1)
 		(exclude_from_sim no)
@@
 		(fields_autoplaced yes)
 		(property "Reference" "#PWR031"
-			(at 115.57 128.27 0)
+			(at 121.92 128.27 0)
 			(effects
 				(font
@@
 		)
 		(property "Value" "GND"
-			(at 115.57 127 0)
+			(at 121.92 127 0)
 			(effects
 				(font
@@
 		)
 		(property "Footprint" ""
-			(at 115.57 121.92 0)
+			(at 121.92 121.92 0)
 			(effects
 				(font
@@
 		)
 		(property "Datasheet" ""
-			(at 115.57 121.92 0)
+			(at 121.92 121.92 0)
 			(effects
 				(font
@@
 		)
 		(property "Description" "Power symbol creates a global label with name \"GND\" , ground"
-			(at 115.57 121.92 0)
+			(at 121.92 121.92 0)
 			(effects
 				(font
@@
 	(symbol
 		(lib_id "power:GND")
-		(at 171.45 118.11 0)
+		(at 167.64 120.65 0)
 		(unit 1)
 		(exclude_from_sim no)
@@
 		(fields_autoplaced yes)
 		(property "Reference" "#PWR032"
-			(at 171.45 124.46 0)
+			(at 167.64 127 0)
 			(effects
 				(font
@@
 		)
 		(property "Value" "GND"
-			(at 171.45 123.19 0)
+			(at 167.64 125.73 0)
 			(effects
 				(font
@@
 		)
 		(property "Footprint" ""
-			(at 171.45 118.11 0)
+			(at 167.64 120.65 0)
 			(effects
 				(font
@@
 		)
 		(property "Datasheet" ""
-			(at 171.45 118.11 0)
+			(at 167.64 120.65 0)
 			(effects
 				(font
@@
 		)
 		(property "Description" "Power symbol creates a global label with name \"GND\" , ground"
-			(at 171.45 118.11 0)
-			(effects
-				(font
+			(at 167.64 120.65 0)
+			(effects
+				(font

Commit message: Working on V2
Parts:
- added J4: Conn_01x02, symbol Connector_Generic:Conn_01x02
- added R31: R_US, symbol Device:R_US
Connections:
- net +3.3V: now also R31.1
- net GND: now also J4.2 (Pin_2)
- net HPFBYPASS renamed ADC_HPFBYPASS
- net ADC_HPFBYPASS: now also J4.1 (Pin_1), R31.2
- net ~{RST} renamed ~{ADC_RST}
Other:
- note added: "HPF enabled by default, can be disabled for testing. NOTE: When HPF is enabled it's not possible to test the ADC with DC levels."

Commit message: First draft of schematic
Other:
- note added: "The TI PCM1804 is a 24-bit stereo analog to digital converter designed for audio applications. It contains an integrated low-pass anti-aliasing filter on the front-end with a cut-off around 20 kHz. Sample rate (f_{s}) will be 48,000 samples/second. Narrower filtering will be achieved in DSP."
- moved on the sheet: C10, C11, C12, C13, C14, C15, C16, C17, C18, C19, L1, U3

Commit message: First draft of schematic
Other:
- note added: "HPF enabled by default, can be disabled for testing using this jumper block. NOTE: When HPF is enabled it's not possible to test the ADC with DC levels."
- note added: "OSR=010, 384*f_{s} by default"
- note removed: "HPF enabled by default, can be disabled for testing. NOTE: When HPF is enabled it's not possible to test the ADC with DC levels."
- note removed: "OSR=010, 384*fs by default"
- moved on the sheet: C10, C11, C12, C13, C14, C15, C16, C17, C18, C19, L1, U3

Commit message: First draft of schematic
Parts:
- R31: value R_US -> 4.7k
Other:
- note added: "Configuration Solder Bridges"
- moved on the sheet: J4, JP10, R31
