File: hw/if-2/adc.kicad_sch (KiCad schematic)
At the start: 20 parts, among them J4 Conn_01x02, U3 PCM1804DBR

Commit message: Ready to do layout on IF2 board
Parts:
- removed C10, C13, C16, C18: 10u, Capacitor_THT:CP_Radial_D4.0mm_P2.00mm, symbol Device:C_Polarized_Small_US
- removed C12, C15: 1u, Capacitor_SMD:C_0805_2012Metric_Pad1.18x1.45mm_HandSolder, symbol Device:C_Polarized_Small_US
- added C10, C12, C15, C16: 1u, Capacitor_SMD:C_0805_2012Metric_Pad1.18x1.45mm_HandSolder, symbol Device:C_Small
- added C13, C18: 10u, Capacitor_SMD:C_0805_2012Metric_Pad1.18x1.45mm_HandSolder, symbol Device:C_Small
- J4: footprint (none) -> Connector_PinHeader_2.54mm:PinHeader_1x02_P2.54mm_Vertical
- R31: footprint (none) -> Resistor_SMD:R_0805_2012Metric_Pad1.20x1.40mm_HandSolder
- U3: footprint DB28 -> Package_SO:SSOP-28_5.3x10.2mm_P0.65mm
Connections:
- net +3.3V: now also C13.1
- net GND: now also C10.2, C12.2, C13.2, C15.2, C16.2, C18.2
- net R0_VCOM: now also C12.1
- net R1_VCOM: now also C15.1
- net VREFL: now also C10.1
- net at C19.1, L1.2, U3.22 (VCC): now also C18.1
- net at C17.1, U3.28 (VREFR): now also C16.1
Other:
- title: Analog To Digital Converter -> COS/CTCSS/PTT Controls (Radio 1)
