File: hw/if-2/audio_out_0.kicad_sch (KiCad schematic)
At the start: 0 parts

Commit message: Working on 2
Parts:
- added C20, C21, C22, C23, C24: 1uF, Capacitor_SMD:C_0805_2012Metric_Pad1.18x1.45mm_HandSolder, symbol Device:C_Small
- added C25: 10uF, Capacitor_SMD:C_0805_2012Metric_Pad1.18x1.45mm_HandSolder, symbol Device:C_Small
- added C26: 0.001uF, Capacitor_SMD:C_0805_2012Metric_Pad1.18x1.45mm_HandSolder, symbol Device:C_Small
- added C9: 100pF, Capacitor_SMD:C_0805_2012Metric_Pad1.18x1.45mm_HandSolder, symbol Device:C_Small
- added R14, R15, R16, R17: 100k, Resistor_SMD:R_0805_2012Metric_Pad1.20x1.40mm_HandSolder, symbol Device:R_Small_US
- added R18: 200k, Resistor_SMD:R_0805_2012Metric_Pad1.20x1.40mm_HandSolder, symbol Device:R_Small_US
- added R19, R21: 10k, Resistor_SMD:R_0805_2012Metric_Pad1.20x1.40mm_HandSolder, symbol Device:R_Small_US
- added R20: 47, Resistor_SMD:R_0805_2012Metric_Pad1.20x1.40mm_HandSolder, symbol Device:R_Small_US
- added RV3: 50k, bruce-footprints:POT_3362P, symbol Device:R_Potentiometer_US
- added TP3: TestPoint, TestPoint:TestPoint_Pad_3.0x3.0mm, symbol Connector:TestPoint
- added U4: LM4562, Package_SO:SOIC-8_3.9x4.9mm_P1.27mm, symbol Amplifier_Operational:LM4562
Connections:
- new net: C22.2, RV3.1, TP3.1
- new net: C9.1, R14.2, R15.2, R16.1, U4.2 (-)
- new net: C22.1, C9.2, R16.2, U4.1
- new net: C20.2, R14.1
- new net: C23.1, R20.1, U4.8 (V+)
- new net: C24.1, RV3.2
- new net: R17.2, R18.1, U4.6 (-)
- new net: C25.1, R18.2, U4.7
- new net: C25.2, R19.1, R21.1
- new net: C21.2, R15.1
- new net: C24.2, R17.1
- new net +2V5: U4.3 (+), U4.5 (+)
- new net +5V: R20.2
- new net GND: C23.2, RV3.3, U4.4 (V-)
- new net RADIO0-TX-N: C26.2, R19.2
- new net RADIO0-TX-P: C26.1, R21.2
- new net TONE: C21.1
- new net TX0-A: C20.1

Commit message: Working on V2
Parts:
- removed C21: 1uF, Capacitor_SMD:C_0805_2012Metric_Pad1.18x1.45mm_HandSolder, symbol Device:C_Small
- removed R15: 100k, Resistor_SMD:R_0805_2012Metric_Pad1.20x1.40mm_HandSolder, symbol Device:R_Small_US
- removed TP3: TestPoint, TestPoint:TestPoint_Pad_3.0x3.0mm, symbol Connector:TestPoint
- C22: value 1uF -> 4.7u
- C23: value 1uF -> 10u
- C24: value 1uF -> 0.47u
- C26: value 0.001uF -> 100p
- C9: value 100pF -> 470p; footprint Capacitor_SMD:C_0805_2012Metric_Pad1.18x1.45mm_HandSolder -> (none)
- R14, R16, R17: value 100k -> 20k
- R18: value 200k -> 68k
- R21: value 10k -> 510
Connections:
- net RADIO0-TX-N is gone; now on net GND: C26.2, R19.2
- net at R14.2, R16.1, U4.2 (-): no longer C9.1
- net at C22.1, R16.2, U4.1: no longer C9.2
- net at R17.2, R18.1, U4.6 (-): now also C9.1
- net at C25.1, R18.2, U4.7: now also C9.2
- net +2V5 renamed VBIAS
- net RADIO0-TX-P renamed R0_AUDIO_OUT
- net TX0-A renamed R0_VOUT
Other:
- note added: "(See page 30 of TI PCM1804 datasheet) https://www.ti.com/lit/ds/symlink/pcm1804.pdf"
- note added: "Approximately 2.5V"
- note added: "Audio output level trim."
- note added: "This is not a pre/de-emphasis filter. That is handled in the DSP."
- note added: "We will use large solder pads and a thru-hole part for this resistor to make it easy to change in the field if the gain is way off."
- title: Digital Repeater Controller  -> Audio Output Processing (Radio 0)
- moved on the sheet: C20, C22, C23, C24, C25, C26, R14, R16, R17, R18, R19, R20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

Commit message: First draft of schematic
Other:
- note added: "(See page 4 of SCOM7K schematic)"
- note removed: "(See page 30 of TI PCM1804 datasheet) https://www.ti.com/lit/ds/symlink/pcm1804.pdf"
Changed lines of the file:
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@@
 		)
 	)
-	(text "(See page 30 of TI PCM1804 datasheet)\n\nhttps://www.ti.com/lit/ds/symlink/pcm1804.pdf\n"
+	(text "(See page 4 of SCOM7K schematic)"
 		(exclude_from_sim no)
 		(at 127 46.482 0)

Commit message: Working on simulation
Parts:
- C24: value 0.47u -> 1u
Changed lines of the file:
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@@
 			)
 		)
-		(property "Value" "0.47u"
+		(property "Value" "1u"
 			(at 132.0863 80.01 90)
 			(effects

Commit message: Simulations
Parts:
- C24: value 1u -> 4.7u
Changed lines of the file:
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@@
 			)
 		)
-		(property "Value" "1u"
+		(property "Value" "4.7u"
 			(at 132.0863 80.01 90)
 			(effects

Commit message: Adding changes suggested by Dan
Parts:
- removed U4: LM4562, Package_SO:SOIC-8_3.9x4.9mm_P1.27mm, symbol Amplifier_Operational:LM4562
- added U4: TL072, symbol Amplifier_Operational:TL072
- C20: value 1uF -> 4.7u
Connections:
- net GND: now also U4.4 (V-)
- net VBIAS: now also U4.3 (+), U4.5 (+)
- net at C23.1, R20.1: now also U4.8 (V+)
- net at R14.2, R16.1: now also U4.2 (-)
- net at C22.1, R16.2: now also U4.1
- net at C9.1, R17.2, R18.1: now also U4.6 (-)
- net at C25.1, C9.2, R18.2: now also U4.7

Commit message: Adding changes suggested by Dan
Parts:
- added C46: 10uF, Capacitor_SMD:C_0805_2012Metric_Pad1.18x1.45mm_HandSolder, symbol Device:C_Small
Connections:
- net R0_AUDIO_OUT: now also C46.2; no longer C26.1, R21.2
- new net: C26.1, C46.1, R21.2
Changed lines of the file:
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@@
 	(wire
 		(pts
-			(xy 196.85 86.36) (xy 207.01 86.36)
+			(xy 196.85 86.36) (xy 212.09 86.36)
 		)
 		(stroke
@@
 		(pts
 			(xy 153.67 58.42) (xy 146.05 58.42)
+		)
+		(stroke
+			(width 0)
+			(type default)
+		)
+	)
+	(wire
+		(pts
+			(xy 217.17 86.36) (xy 223.52 86.36)
 		)
 		(stroke
@@
 	(global_label "R0_AUDIO_OUT"
 		(shape input)
-		(at 207.01 86.36 0)
+		(at 223.52 86.36 0)
 		(fields_autoplaced yes)
 		(effects
@@
 		)
 		(property "Intersheetrefs" "${INTERSHEET_REFS}"
-			(at 223.6629 86.36 0)
+			(at 240.1729 86.36 0)
 			(effects
 				(font
@@
 					(unit 1)
 				)
+			)
+		)
+	)
+	(symbol
+		(lib_id "Device:C_Small")
+		(at 214.63 86.36 90)
+		(unit 1)
+		(exclude_from_sim no)
+		(in_bom yes)
+		(on_board yes)
+		(dnp no)
+		(fields_autoplaced yes)
+		(property "Reference" "C46"
+			(at 214.6363 80.01 90)
+			(effects
+				(font
+					(size 1.27 1.27)
+				)
+			)
+		)
+		(property "Value" "10uF"
+			(at 214.6363 82.55 90)
+			(effects
+				(font
+					(size 1.27 1.27)
+				)
+			)
+		)
+		(property "Footprint" "Capacitor_SMD:C_0805_2012Metric_Pad1.18x1.45mm_HandSolder"
+			(at 214.63 86.36 0)
+			(effects
+				(font
+					(size 1.27 1.27)
+				)
+				(hide yes)
+			)
+		)
+		(property "Datasheet" "~"
+			(at 214.63 86.36 0)
+			(effects
+				(font
+					(size 1.27 1.27)
+				)
+				(hide yes)
+			)
+		)
+		(property "Description" "Unpolarized capacitor, small symbol"
+			(at 214.63 86.36 0)
+			(effects
+				(font
+					(size 1.27 1.27)
+				)
+				(hide yes)
+			)
+		)
+		(pin "1"
+		)
+		(pin "2"
+		)
+		(instances
+			(project "if-2"
+				(path "/a8c2d6aa-29bb-49bd-a367-0d62a0a32480/44344ba6-1370-4a77-ab96-dbf60268a0b4"
+					(reference "C46")
+					(unit 1)
+				)

Commit message: Adding changes suggested by Dan
Parts:
- added C47: 0.1u, Capacitor_SMD:C_0805_2012Metric_Pad1.18x1.45mm_HandSolder, symbol Device:C_Small
Connections:
- net GND: now also C47.2
- net at C23.1, R20.1, U4.8 (V+): now also C47.1
Other:
- moved on the sheet: C23, R20, U4C
