File: hw/if-2/audio_in_0.kicad_sch (KiCad schematic)
At the start: 24 parts, among them U1 LM4562, U2 LM4562

Commit message: Working on V2
Parts:
- added TP2, TP3: TestPoint, symbol Connector:TestPoint
- C5, C6: value 1uF -> 10u
Connections:
- net R0_AUDIO_IN: now also D2.3 (COM), RV1.1
- net R0_VIN+: now also TP3.1
- net R0_VIN-: now also TP2.1
- net R0_VBIAS renamed VBIAS
Other:
- note added: "Approximately 2.5V"
- note added: "Approximately 2.5V center voltage from ADC."
- note added: "Audio input level trim. Adjust attenuation for ADC full-scale."
- note added: "This is not a pre/de-emphasis filter. That is handled in the DSP."
- note added: "We will use large solder pads and a thru-hole part for this resistor to make it easy to change in the field if the gain is way off."
- note removed: "Audio input level trim. Adjust for ADC full-scale."

Commit message: First draft of schematic
Other:
- note added: "Differential audio signal centered at +2.5V"
- moved on the sheet: C1, D2, R1, R3, RV1, U1A

Commit message: First draft of schematic
Other:
- note added: "Audio input from radio"
Changed lines of the file:
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@@
+		)
+	)
+	(text "Audio input from radio"
+		(exclude_from_sim no)
+		(at 73.66 39.624 0)
+		(effects
+			(font
+				(size 1.27 1.27)
+			)
 		)
 	)

Commit message: Simulations
Parts:
- C1: value 0.47u -> 4.7u
- R3: value 100k -> 47k
Other:
- note added: "Audio input from radio. Expected to be in the 100-1000mVpp range."
- note removed: "Audio input from radio"
Changed lines of the file:
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@@
 		)
 	)
-	(text "Audio input from radio"
+	(text "Audio input from radio. \nExpected to be in the 100-1000mVpp range."
 		(exclude_from_sim no)
-		(at 73.66 39.624 0)
+		(at 73.66 43.18 0)
 		(effects
 			(font
@@
 			)
 		)
-		(property "Value" "0.47u"
+		(property "Value" "4.7u"
 			(at 134.6136 41.91 90)
 			(effects
@@
 			)
 		)
-		(property "Value" "100k"
+		(property "Value" "47k"
 			(at 166.37 33.02 90)
 			(effects

Commit message: Adding changes suggested by Dan
Parts:
- removed D2: BAT54S, Package_TO_SOT_SMD:SOT-23, symbol Diode:BAT54S
- removed U1, U2: LM4562, Package_SO:SOIC-8_3.9x4.9mm_P1.27mm, symbol Amplifier_Operational:LM4562
- added C42: 4.7u, symbol Device:C_Small
- added C43, C44: 01.u, symbol Device:C_Small
- added C45: 0.001u, symbol Device:C_Small
- added R36, R37: 1k, symbol Device:R_US
- added U1, U2: TL072, symbol Amplifier_Operational:TL072
Connections:
- net GND: now also C43.2, C44.2, C45.2, U1.4 (V-), U2.4 (V-)
- net R0_AUDIO_IN: now also C42.1; no longer RV1.1
- net R0_VCOM: now also U2.3 (+), U2.5 (+)
- net VBIAS: now also U1.3 (+), U1.5 (+)
- net at R5.2, R7.1: now also U1.6 (-)
- net at C3.1, R7.2: now also U1.7
- net at C6.1, R12.2: now also C44.1, U2.8 (V+)
- net at C4.1, R13.2, R8.1: now also U2.6 (-)
- net at C4.2, R10.1: now also U2.7
- net at C5.1, R11.2: now also C43.1, U1.8 (V+)
- net at C2.1, R2.2, R4.1: now also U2.2 (-)
- net at R1.2, R3.1: now also U1.2 (-)
- net at C2.2, R6.1: now also U2.1
- net R0_AUDIO_IN_B: no longer names the net of C7.1, R5.1
- net R0_AUDIO_IN_B: now also R36.2; no longer R3.2
- new net: C42.2, R37.1
- new net: C45.1, R37.2, RV1.1
- new net: R3.2, R36.1, U1.1
Other:
- note added: "AC-coupled audio input from radio. Expected to be in the 100-1000mVpp range."
- note added: "Op Amp Supply Filter"
- note added: "RFI Filter"
- note removed: "Audio input from radio. Expected to be in the 100-1000mVpp range."
- note removed: "Overvoltage protection"
- moved on the sheet: C5, C6, R11, R12

Commit message: Docs
Parts:
- C3, C7: value 10u -> 4.7u
- R3: value 47k -> 100k
Changed lines of the file:
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@@
 			)
 		)
-		(property "Value" "47k"
+		(property "Value" "100k"
 			(at 166.37 33.02 90)
 			(effects
@@
 			)
 		)
-		(property "Value" "10u"
+		(property "Value" "4.7u"
 			(at 130.8163 144.78 90)
 			(effects
@@
 			)
 		)
-		(property "Value" "10u"
+		(property "Value" "4.7u"
 			(at 130.8163 100.33 90)
 			(effects
