File: hw/if-2/if-2.kicad_sch (KiCad schematic)
At the start: 2 parts, among them J1 DB25_Socket, J2 PJ-102AH

Commit message: Working on V2
Parts:
- added H1, H2, H3, H4: MountingHole, symbol Mechanical:MountingHole
- added J3: Conn_02x12_Top_Bottom, symbol Connector_Generic:Conn_02x12_Top_Bottom
Connections:
- net +12V: now also J3.21 (Pin_21); no longer J2.1
- net GND: now also J3.12 (Pin_12), J3.24 (Pin_24)
- net R0_COR renamed R0_COS
- net R1_COR renamed R1_COS
- new net +3.3V: J3.23 (Pin_23)
- new net +5V: J3.22 (Pin_22)
- new net 12V_UNFUSED: J2.1
- new net ADC_BCK: J3.3 (Pin_3)
- new net ADC_DOUT: J3.4 (Pin_4)
- new net ADC_LRCK: J3.2 (Pin_2)
- new net ADC_SCK: J3.1 (Pin_1)
- new net DAC_BCK: J3.7 (Pin_7)
- new net DAC_DIN: J3.8 (Pin_8)
- new net DAC_LRCK: J3.6 (Pin_6)
- new net DAC_SCK: J3.5 (Pin_5)
- new net R0_COS_B: J3.14 (Pin_14)
- new net R0_CTCSS_B: J3.16 (Pin_16), J3.17 (Pin_17)
- new net R0_PTT_B: J3.18 (Pin_18)
- new net R1_COS_B: J3.15 (Pin_15)
- new net R1_PTT_B: J3.19 (Pin_19)
- new net ~{ADC_RST}: J3.13 (Pin_13)
- no-connect marks 11 -> 16
Other:
- added sheet Audio Out 1 (audio_out_1.kicad_sch)
- added sheet DAC (dac.kicad_sch)
- added sheet Power (power.kicad_sch)
- note added: "Ribbon cable to digital module"

Commit message: First draft of schematic
Parts:
- removed J1: DB25_Socket, symbol Connector:DB25_Socket
- removed J2: PJ-102AH, bruce-footprints:Power_5.5mm_CUI_PJ-102AH, symbol symbol-library-1:Power_5.5mm_PJ-102AH
- removed J3: Conn_02x12_Top_Bottom, symbol Connector_Generic:Conn_02x12_Top_Bottom
Connections:
- no-connect marks 16 -> 0
Other:
- added sheet Connectors (connectors.kicad_sch)
- note added: "Copyright (C) Bruce MacKinnon KC1FSZ, 2025 This design is licensed under the terms of the TAPR Open Hardware License (OHL) and is intended for AMATEUR RADIO USE ONLY. Commercial use of this design is prohibited."
- note added: "Digital Repeater Controller V2"
- note added: "NOTES: * This is an analog board that interfaces with two radios. A separate digital board based on the RP2040 is also required. A ribbon cable connects the two boards. * The goal of this design is to do as little as possible in hardware. * Many things that usually happen in hardware (or FPGA) will happen in software: - Audio routing between the two radios will happen in software. - Audio pre-emp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"
- note removed: "5.5mm Power Connector +12V on center pin"
- note removed: "DB25 Female (Equivalent to J2 on SCOM7K)"
- note removed: "Ribbon cable to digital module"
- moved on the sheet: H1, H2, H3, H4

Commit message: Adding changes suggested by Dan
Other:
- sheet Controls renamed Controls 0
- added sheet Controls 1 (controls_1.kicad_sch)
- sheet Controls 0: file controls.kicad_sch -> controls_0.kicad_sch
Changed lines of the file:
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@@
+	)
+	(sheet
+		(at 213.36 109.22)
+		(size 24.13 22.86)
+		(exclude_from_sim no)
+		(in_bom yes)
+		(on_board yes)
+		(dnp no)
+		(fields_autoplaced yes)
+		(stroke
+			(width 0.1524)
+			(type solid)
+		)
+		(fill
+			(color 0 0 0 0.0000)
+		)
+		(property "Sheetname" "Controls 1"
+			(at 213.36 108.5084 0)
+			(effects
+				(font
+					(size 1.27 1.27)
+				)
+				(justify left bottom)
+			)
+		)
+		(property "Sheetfile" "controls_1.kicad_sch"
+			(at 213.36 132.6646 0)
+			(effects
+				(font
+					(size 1.27 1.27)
+				)
+				(justify left top)
+			)
+		)
+		(instances
+			(project "if-2"
+				(path "/a8c2d6aa-29bb-49bd-a367-0d62a0a32480"
+					(page "10")
+				)
+			)
+		)
 	)
 	(sheet
@@
 	)
 	(sheet
-		(at 217.17 109.22)
+		(at 62.865 142.24)
 		(size 22.86 22.86)
 		(exclude_from_sim no)
@@
 		)
 		(property "Sheetname" "Power"
-			(at 217.17 108.5084 0)
+			(at 62.865 141.5284 0)
 			(effects
 				(font
@@
 		)
 		(property "Sheetfile" "power.kicad_sch"
-			(at 217.17 132.6646 0)
-			(effects
-				(font
-					(size 1.27 1.27)
-				)
-				(justify left top)
-			)
-		)
-		(instances
-			(project "if-2"
-				(path "/a8c2d6aa-29bb-49bd-a367-0d62a0a32480"
-					(page "10")
+			(at 62.865 165.6846 0)
+			(effects
+				(font
+					(size 1.27 1.27)
+				)
+				(justify left top)
+			)
+		)
+		(instances
+			(project "if-2"
+				(path "/a8c2d6aa-29bb-49bd-a367-0d62a0a32480"
+					(page "11")
 				)
 			)
@@
 			(color 0 0 0 0.0000)
 		)
-		(property "Sheetname" "Controls"
+		(property "Sheetname" "Controls 0"
 			(at 186.69 108.5084 0)
 			(effects
@@
 			)
 		)
-		(property "Sheetfile" "controls.kicad_sch"
+		(property "Sheetfile" "controls_0.kicad_sch"
 			(at 186.69 132.6646 0)
 			(effects

Commit message: Docs
Other:
- note added: "Digital Repeater Controller V2 - Radio Interface Board"
- note removed: "Digital Repeater Controller V2"
Changed lines of the file:
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@@
 		)
 	)
-	(text "Digital Repeater Controller V2"
+	(text "Digital Repeater Controller V2 - Radio Interface Board"
 		(exclude_from_sim no)
-		(at 47.244 21.844 0)
+		(at 71.374 21.082 0)
 		(effects
 			(font
@@
 		)
 	)
-	(text "NOTES:\n* This is an analog board that interfaces with two radios. A separate digital board based on the RP2040 is also required. A ribbon cable\n  connects the two boards.\n* The goal of this design is to do as little as possible in hardware.\n* Many things that usually happen in hardware (or FPGA) will happen in software:\n  - Audio routing between the two radios will happen in software.\n  - Audio pre-emphasis/de-emphasis (if needed) will happen using DSP using digital filters.\n  - CTCSS decoding (if needed) will happen in DSP.\n  - CTCSS encoding (if needed) will happen in DSP.\n  - DTMF decoding will happen in DSP.\n  - CWID and other tone prompts will happen in DSP/software.\n  - Voice IDs will happen in DSP/software.\n\n"
+	(text "NOTES:\n* This is an analog board that interfaces with two radios. A separate digital board based on the RP2040 is also required. A ribbon cable\n  connects the two boards.\n* The goal of this design is to do as little as possible in hardware.\n* Many things that usually happen in hardware (or FPGA) will happen in software:\n  - Audio routing between the two radios will happen in software.\n  - Audio pre-emphasis/de-emphasis (if needed) will happen using DSP using digital filters.\n  - CTCSS decoding (if needed) will happen in DSP.\n  - CTCSS encoding (if needed) will happen in DSP.\n  - DTMF decoding will happen in DSP.\n  - CWID and other tone prompts will happen in DSP/software.\n  - Voice IDs will happen in DSP/software.\n  - Other digital audio interfaces like EchoLink (or DMR/D-Star in the future) will be directly integrated.\n\n"
 		(exclude_from_sim no)
 		(at 18.034 49.276 0)

Commit message: Ready to do layout on IF2 board
Parts:
- H1, H2, H3, H4: footprint (none) -> MountingHole:MountingHole_3.5mm
Other:
- title: Digital Repeater Controller  -> COS/CTCSS/PTT Controls (Radio 1)
Changed lines of the file:
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@@
 	(paper "USLetter")
 	(title_block
-		(title "Digital Repeater Controller ")
+		(title "COS/CTCSS/PTT Controls (Radio 1)")
 		(date "2025-03-18")
 		(rev "2")
@@
 			)
 		)
-		(property "Footprint" ""
+		(property "Footprint" "MountingHole:MountingHole_3.5mm"
 			(at 133.35 186.69 0)
 			(effects
@@
 			)
 		)
-		(property "Footprint" ""
+		(property "Footprint" "MountingHole:MountingHole_3.5mm"
 			(at 133.35 180.34 0)
 			(effects
@@
 			)
 		)
-		(property "Footprint" ""
+		(property "Footprint" "MountingHole:MountingHole_3.5mm"
 			(at 133.35 193.04 0)
 			(effects
@@
 			)
 		)
-		(property "Footprint" ""
+		(property "Footprint" "MountingHole:MountingHole_3.5mm"
 			(at 133.35 173.99 0)
 			(effects

Commit message: Making progress on layout
Other:
- title: COS/CTCSS/PTT Controls (Radio 1) -> Title Page
Changed lines of the file:
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@@
 	(paper "USLetter")
 	(title_block
-		(title "COS/CTCSS/PTT Controls (Radio 1)")
-		(date "2025-03-18")
+		(title "Title Page")
+		(date "2025-05-09")
 		(rev "2")
 		(company "Bruce MacKinnon KC1FSZ")
