File: hw/if-2/if-2.kicad_sch (KiCad schematic)
At the start: 4 parts

Commit message: Layout passes DRC!!
Other:
- title: Title Page -> Digital Repeater Controller
Changed lines of the file:
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@@
 	(paper "USLetter")
 	(title_block
-		(title "Title Page")
+		(title "Digital Repeater Controller")
 		(date "2025-05-09")
 		(rev "2")
