File: hw/if-2/power.kicad_sch (KiCad schematic)
At the start: 21 parts, among them J5 Conn_01x02, U10 NCP1117-5.0_SOT223, U11 NCP1117-3.3_SOT223

Commit message: Progress on layout
Parts:
- C41: footprint Capacitor_THT:CP_Radial_D5.0mm_P2.50mm -> Capacitor_THT:CP_Radial_D7.5mm_P2.50mm
Changed lines of the file:
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@@
 			)
 		)
-		(property "Footprint" "Capacitor_THT:CP_Radial_D5.0mm_P2.50mm"
+		(property "Footprint" "Capacitor_THT:CP_Radial_D7.5mm_P2.50mm"
 			(at 185.42 99.06 0)
 			(effects
