File: hw/if-2/if-2.kicad_pcb (KiCad board)
At the start: 2 copper layers, 193 parts, among them J1 DB25_Socket, J2 PJ-102AH, J3 Conn_02x12_Odd_Even, J4 Conn_01x02, J5 Conn_01x02, Q1 MMBT3904, Q11 MMBT3904, Q12 MMBT3904, Q2 MMBT3904, U10 NCP1117-5.0_SOT223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

Commit message: Making progress on layout
Parts:
- moved TP61 19.4 mm to (193.0, 117.8), turned to -90 degrees
- moved TP41 19.1 mm to (192.0, 89.0), turned to -90 degrees
- moved TP62 17.8 mm to (193.0, 125.8), turned to -90 degrees
- moved C52 17.6 mm to (192.2, 93.0), turned to 90 degrees
- moved C68 17.4 mm to (192.8, 121.7), turned to 90 degrees
- moved TP42 16.8 mm to (191.8, 97.0), turned to -90 degrees
- moved R67 15.6 mm to (190.0, 117.8), turned to 90 degrees
- moved R47 15.2 mm to (188.8, 89.0), turned to 90 degrees
- moved R45 14.1 mm to (174.2, 89.2), turned to -90 degrees
- moved R68 13.6 mm to (190.0, 125.8), turned to -90 degrees
- moved R70 13.1 mm to (187.8, 117.8), turned to 90 degrees
- moved R65 12.8 mm to (175.8, 118.8), turned to -90 degrees
- moved R50 12.7 mm to (186.5, 89.0), turned to 90 degrees
- moved R48 12.5 mm to (188.8, 96.8), turned to -90 degrees
- moved C45 11.9 mm to (172.0, 89.2), turned to 90 degrees
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Connections:
- R42 pad 1: Net-(C49-Pad1) -> Net-(C45-Pad1)
- R43 pad 2: Net-(C45-Pad1) -> Net-(C49-Pad1)
- R52 pad 2: Net-(C49-Pad1) -> Net-(C45-Pad1)
- R62 pad 1: Net-(C65-Pad1) -> Net-(C64-Pad1)
- R63 pad 2: Net-(C64-Pad1) -> Net-(C65-Pad1)
- R72 pad 2: Net-(C65-Pad1) -> Net-(C64-Pad1)
- U41 pad 7: Net-(C45-Pad1) -> Net-(C49-Pad1)
- U61 pad 7: Net-(C64-Pad1) -> Net-(C65-Pad1)
Routing:
- net Net-(U62B--): track 0.00 -> 19.1 mm
- net Net-(U62A--): track 0.00 -> 18.7 mm
- net Net-(C65-Pad1): track 0.00 -> 18.5 mm
- net Net-(C64-Pad1): track 0.00 -> 17.3 mm
- net Net-(D61-COM): track 0.00 -> 16.3 mm
- net Net-(R69-Pad2): track 0.00 -> 10.1 mm
- net R1_VIN+: track 0.00 -> 8.77 mm
- net R1_VIN-: track 0.00 -> 8.69 mm
- net Net-(C67-Pad2): track 0.00 -> 8.68 mm
- net Net-(C49-Pad1): track 7.35 -> 15.5 mm
- net Net-(C62-Pad1): track 0.00 -> 7.82 mm
- net Net-(U61B--): track 0.00 -> 7.11 mm
- net VBIAS: track 5.48 -> 11.0 mm
- net Net-(C66-Pad2): track 0.00 -> 5.41 mm
- net Net-(C63-Pad2): track 0.00 -> 5.02 mm
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Other:
- copper layers 2 -> 4

Commit message: Making progress on layout
Parts:
- moved J3 224.2 mm to (251.7, 84.9)
- moved C81 176.4 mm to (198.2, 112.8), turned to 180 degrees
- moved C82 175.4 mm to (198.2, 119.8)
- moved C88 172.8 mm to (189.8, 119.2)
- moved R82 171.4 mm to (198.2, 117.5), turned to 180 degrees
- moved R81 171.2 mm to (198.2, 115.0)
- moved C87 171.1 mm to (189.8, 121.4)
- moved C84 167.1 mm to (185.8, 112.8), turned to -90 degrees
- moved R54 165.5 mm to (183.5, 73.0)
- moved R87 164.8 mm to (189.8, 123.6)
- moved U81 164.6 mm to (191.5, 114.6), turned to 180 degrees
- moved C56 162.1 mm to (183.5, 68.5), turned to 180 degrees
- moved C85 161.8 mm to (179.0, 112.8), turned to -90 degrees
- moved C86 160.8 mm to (176.8, 112.8), turned to -90 degrees
- moved R85 160.4 mm to (183.5, 112.8), turned to 90 degrees
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Connections:
- J3 pad 11: DAC_LRCK -> DAC_DIN
- J3 pad 15: DAC_DIN -> DAC_SCK
- J3 pad 9: DAC_SCK -> DAC_LRCK
Routing:
- net Net-(C92-Pad2): track 0.00 -> 19.6 mm
- net Net-(C82-Pad2): track 0.00 -> 19.5 mm
- net Net-(U81B--): track 0.00 -> 15.8 mm
- net Net-(C64-Pad1): track 17.3 -> 30.9 mm
- net +3.3V: track 0.00 -> 11.9 mm
- net VBIAS: track 11.0 -> 21.9 mm
- net Net-(C94-Pad1): track 0.00 -> 10.7 mm
- net Net-(U81A--): track 0.00 -> 8.51 mm
- net Net-(U41C-V+): track 0.00 -> 8.33 mm
- net Net-(U61C-V+): track 0.00 -> 8.22 mm
- net Net-(U91A--): track 0.00 -> 8.06 mm
- net Net-(U42C-V+): track 0.00 -> 7.58 mm
- net Net-(U91B--): track 0.00 -> 7.52 mm
- net Net-(U62C-V+): track 0.00 -> 7.51 mm
- net Net-(C45-Pad1): track 16.8 -> 24.0 mm
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
Commit message: Making progress on layout
Parts:
- added TP10: TestPoint, TestPoint:TestPoint_Pad_2.5x2.5mm, F.Cu at (56.0, 143.0)
- added TP6: TestPoint, TestPoint:TestPoint_Pad_2.5x2.5mm, F.Cu at (86.2, 72.0)
- added TP7: TestPoint, TestPoint:TestPoint_Pad_2.5x2.5mm, F.Cu at (86.0, 98.2)
- added TP8: TestPoint, TestPoint:TestPoint_Pad_2.5x2.5mm, F.Cu at (85.2, 140.2)
- added TP9: TestPoint, TestPoint:TestPoint_Pad_2.5x2.5mm, F.Cu at (85.2, 144.5)
- moved C27 127.3 mm to (113.6, 72.6)
- moved C32 127.3 mm to (118.0, 76.6)
- moved C33 127.3 mm to (101.8, 83.6)
- moved JP1 127.3 mm to (119.2, 89.0)
- moved JP2 127.3 mm to (119.2, 83.0)
- moved JP3 127.3 mm to (114.3, 86.0)
- moved JP4 127.3 mm to (119.2, 86.0)
- moved R15 127.3 mm to (101.8, 76.6)
- moved U5 127.3 mm to (110.8, 78.6)
- moved C31 127.3 mm to (110.0, 85.2)
- moved C21 127.3 mm to (107.8, 72.2)
- moved C28 127.3 mm to (101.8, 72.0)
- moved C29 127.3 mm to (107.8, 85.2)
- moved C30 127.3 mm to (101.8, 74.2)
- moved C34 127.3 mm to (101.8, 78.8)
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- renumbered TP41 to TP2, TP42 to TP3, TP61 to TP4, TP62 to TP5
Routing:
- removed copper zone on F.Cu, net GND
Other:
- board outline added: 100 x 129 mm
- board text added: "KC1FSZ bruce@mackinnon.com"
- board text added: "R0 In Lvl"
- board text added: "R0 Out Lvl"
- board text added: "R1 In Lvl"
- board text added: "R1 Out Lvl"
- board text added: "V2 2025-05 B"
- board text added: "W1TKZ Digital Repeater Controller"

Commit message: Workig on routing
Parts:
- moved J5 34.3 mm to (55.1, 119.5), turned to 0 degrees
- moved CR11 34.0 mm to (50.8, 125.2)
- moved C41 34.0 mm to (44.4, 119.2)
- moved D9 34.0 mm to (50.9, 120.0)
- moved TP9 29.5 mm to (56.0, 140.8)
- moved JP2 9.51 mm to (119.5, 73.5), turned to 180 degrees
- moved JP4 9.50 mm to (119.5, 76.5)
- moved C32 8.47 mm to (110.8, 72.3), turned to 90 degrees
- moved C15 5.00 mm to (125.6, 58.0)
- moved C16 5.00 mm to (130.0, 58.0)
- moved C17 5.00 mm to (127.8, 58.0)
- moved C18 5.00 mm to (120.2, 57.9)
- moved C19 5.00 mm to (122.4, 57.9)
- moved L1 5.00 mm to (118.0, 57.9)
- moved JP1 3.06 mm to (119.8, 86.0)
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Routing:
- net GND: track 0.00 -> 214.2 mm, vias 0 -> 55
- net +3.3V: track 11.9 -> 95.2 mm, vias 0 -> 9
- net +12V: track 0.00 -> 44.8 mm
- net ADC_DOUT: track 0.00 -> 36.0 mm
- net +5V: track 0.00 -> 35.7 mm
- net ADC_BCK: track 0.00 -> 33.8 mm
- net ADC_LRCK: track 0.00 -> 31.5 mm
- net ~{ADC_RST}: track 0.00 -> 30.0 mm
- net ADC_SCK: track 0.00 -> 29.1 mm
- net DAC_SCK: track 0.00 -> 21.3 mm
- net DAC_BCK: track 0.00 -> 21.0 mm
- net FMT0: track 0.00 -> 20.5 mm
- net DAC_LRCK: track 0.00 -> 20.2 mm
- net DAC_DIN: track 0.00 -> 19.7 mm
- net FMT1: track 0.00 -> 19.4 mm
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- added copper zone on In1.Cu, net GND
Other:
- board size 100 x 129 mm -> 100 x 130 mm

Commit message: Workig on routing
Parts:
- moved C41 11.2 mm to (53.3, 112.5), turned to 180 degrees
- moved CR11 7.23 mm to (47.2, 118.9), turned to -90 degrees
- moved J5 4.39 mm to (53.0, 123.3), turned to -90 degrees
- moved J2 2.70 mm to (47.5, 130.8)
- moved D9 1.82 mm to (52.4, 119.0), turned to 90 degrees
Routing:
- net +12V: track 44.8 -> 35.3 mm
- net 12V_UNFUSED: track 11.9 -> 8.99 mm

Commit message: Progress on layout
Parts:
- C41: footprint Capacitor_THT:CP_Radial_D5.0mm_P2.50mm -> Capacitor_THT:CP_Radial_D7.5mm_P2.50mm
- moved TP1 40.8 mm to (44.4, 137.9)
- moved TP9 30.0 mm to (86.0, 140.0)
- moved TP8 20.6 mm to (65.0, 144.0)
- moved C35 19.0 mm to (57.0, 141.0)
- moved D1 18.8 mm to (78.8, 140.0)
- moved R28 18.8 mm to (81.0, 140.0)
- moved C38 17.4 mm to (77.2, 125.5)
- moved C40 17.4 mm to (79.8, 125.5)
- moved U11 17.4 mm to (80.0, 132.8)
- moved TP10 17.2 mm to (71.0, 136.0)
- moved D8 14.3 mm to (64.3, 140.2)
- moved C39 9.40 mm to (61.8, 125.8)
- moved U10 9.40 mm to (62.0, 133.1)
- moved C37 9.40 mm to (59.2, 125.8)
- moved C36 9.10 mm to (73.0, 144.0), turned to -90 degrees
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Connections:
- U62 pad 3: R0_VCOM -> R1_VCOM
- U62 pad 5: R0_VCOM -> R1_VCOM
Routing:
- net +5V: track 35.7 -> 262.7 mm, vias 0 -> 12
- net +12V: track 35.3 -> 194.1 mm
- net R0_AUDIO_IN: track 0.00 -> 83.3 mm, vias 0 -> 1
- net R0_VCOM: track 4.02 -> 59.1 mm, vias 0 -> 3
- net R1_VCOM: track 7.92 -> 59.4 mm, vias 0 -> 3
- net R1_AUDIO_IN: track 0.00 -> 44.8 mm
- net R0_VIN-: track 8.96 -> 39.8 mm, vias 0 -> 2
- net R0_VIN+: track 8.75 -> 36.5 mm, vias 0 -> 2
- net R0_AUDIO_OUT: track 0.00 -> 26.7 mm
- net R1_VOUT: track 0.00 -> 26.6 mm
- net R1_VIN+: track 8.77 -> 32.9 mm, vias 0 -> 2
- net R1_AUDIO_OUT: track 0.00 -> 22.9 mm
- net R0_VOUT: track 0.00 -> 22.2 mm
- net R1_VIN-: track 8.69 -> 28.0 mm
- net Net-(U91B--): track 7.52 -> 17.8 mm
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- added copper zone on In2.Cu, net +3.3V
- added copper zone on In2.Cu, net +5V

Commit message: Layout passes DRC!!
Parts:
- moved H1 1.00 mm to (43.0, 22.0)
- moved H2 1.00 mm to (135.0, 22.0)
- moved H3 1.00 mm to (43.0, 144.0)
- moved H4 1.00 mm to (135.0, 144.0)
Connections:
- J3 pad 10: R1_CTCSS_B -> R1_PTT_B
- J3 pad 12: R0_PTT_B -> R1_CTCSS_B
- J3 pad 14: R1_PTT_B -> R1_COS_B
- J3 pad 4: R0_COS_B -> R0_PTT_B
- J3 pad 6: R1_COS_B -> R0_CTCSS_B
- J3 pad 8: R0_CTCSS_B -> R0_COS_B
Routing:
- net R1_COS: track 4.40 -> 120.1 mm, vias 0 -> 1
- net VBIAS: track 33.4 -> 146.0 mm, vias 0 -> 8
- net R0_COS: track 4.20 -> 110.3 mm, vias 0 -> 2
- net R1_PTT: track 1.94 -> 97.9 mm, vias 0 -> 4
- net R1_CTCSS: track 4.20 -> 94.6 mm, vias 0 -> 2
- net R0_CTCSS: track 4.20 -> 82.3 mm, vias 0 -> 2
- net R1_PTT_B: track 0.00 -> 73.5 mm, vias 0 -> 1
- net R1_CTCSS_B: track 2.80 -> 66.7 mm, vias 0 -> 1
- net R0_PTT: track 2.17 -> 64.7 mm, vias 0 -> 2
- net R0_PTT_B: track 0.00 -> 61.0 mm, vias 0 -> 1
- net R0_COS_B: track 3.40 -> 61.4 mm, vias 0 -> 1
- net R0_CTCSS_B: track 2.80 -> 58.8 mm, vias 0 -> 1
- net R1_COS_B: track 3.00 -> 58.2 mm, vias 0 -> 1
- net +3.3V: track 102.1 -> 108.0 mm, vias 16 -> 17
- net Net-(C64-Pad1): track 30.9 -> 26.4 mm
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
Commit message: Layout passes DRC!!
Routing:
- net GND: track 224.3 -> 232.0 mm, vias 64 -> 83
- added copper zone on F.Cu, net GND
Changed lines of the file:
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@@
 		(legacy_teardrops no)
 	)
-	(paper "A4")
+	(paper "USLetter")
+	(title_block
+		(title "Digital Repeater Controller")
+		(date "2025-05-11")
+		(rev "1")
+		(company "Bruce MacKinnon KC1FSZ")
+		(comment 1 "Copyright (C) 2025, Bruce MacKinnon")
+		(comment 2 "NOT FOR COMMERCIAL USE")
+	)
 	(layers
 		(0 "F.Cu" signal)
@@
 	)
 	(segment
+		(start 64.9625 102.2)
+		(end 64.9625 102.9625)
+		(width 0.2)
+		(layer "F.Cu")
+		(net 2)
+	)
+	(segment
 		(start 65.525 35.955)
 		(end 62.6776 35.955)
@@
 	)
 	(segment
+		(start 64.75 76.25)
+		(end 63 78)
+		(width 0.2)
+		(layer "F.Cu")
+		(net 2)
+	)
+	(segment
 		(start 127.8 59)
 		(end 130 59)
@@
 	)
 	(segment
+		(start 64.9625 102.9625)
+		(end 66 104)
+		(width 0.2)
+		(layer "F.Cu")
+		(net 2)
+	)
+	(segment
 		(start 76.575 81.5)
 		(end 76.575 83.6)
@@
 	)
 	(segment
+		(start 64.75 76.0375)
+		(end 64.75 76.25)
+		(width 0.2)
+		(layer "F.Cu")
+		(net 2)
+	)
+	(segment
 		(start 95.25 100.1)
 		(end 95.6 100.1)
@@
 	)
 	(segment
+		(start 48.29325 73.29325)
+		(end 49 74)
+		(width 0.2)
+		(layer "F.Cu")
+		(net 2)
+	)
+	(segment
 		(start 119.4 100.4)
 		(end 121.4 100.4)
@@
 	)
 	(segment
+		(start 47.8925 73.29325)
+		(end 48.29325 73.29325)
+		(width 0.2)
+		(layer "F.Cu")
+		(net 2)
+	)
+	(segment
 		(start 127.8 100.525)
 		(end 129.475 100.525)
@@
 	)
 	(segment
+		(start 59 53)
+		(end 60 52)
+		(width 0.2)
+		(layer "F.Cu")
+		(net 2)
+	)
+	(segment
 		(start 106.4 120.2)
 		(end 104.7 120.2)
@@
 	)
 	(via
+		(at 60 52)
+		(size 0.6)
+		(drill 0.3)
+		(layers "F.Cu" "B.Cu")
+		(net 2)
+	)
+	(via
 		(at 81.65 124.3)
 		(size 0.6)
@@
 	)
 	(via
+		(at 49 74)
+		(size 0.6)
+		(drill 0.3)
+		(layers "F.Cu" "B.Cu")
+		(net 2)
+	)
+	(via
 		(at 99.25 75.25)
 		(size 0.6)
@@
 	)
 	(via
+		(at 111 45)
+		(size 0.6)
+		(drill 0.3)
+		(layers "F.Cu" "B.Cu")
+		(free yes)
+		(net 2)
+	)
+	(via
+		(at 44 131)
+		(size 0.6)
+		(drill 0.3)
+		(layers "F.Cu" "B.Cu")
+		(free yes)
+		(net 2)
+	)
+	(via
 		(at 121 119.5)
 		(size 0.6)
@@
 	)
 	(via
+		(at 128 67)
+		(size 0.6)
+		(drill 0.3)
+		(layers "F.Cu" "B.Cu")
+		(free yes)
+		(net 2)
+	)
+	(via
 		(at 69.5 49.25)
 		(size 0.6)
@@
 	)
 	(via
+		(at 66 104)
+		(size 0.6)
+		(drill 0.3)
+		(layers "F.Cu" "B.Cu")
+		(net 2)
+	)
+	(via
 		(at 117 86)
 		(size 0.6)
@@
 	)
 	(via
+		(at 134 123)
+		(size 0.6)
+		(drill 0.3)
+		(layers "F.Cu" "B.Cu")
+		(free yes)
+		(net 2)
+	)
+	(via
 		(at 49 120.5)
 		(size 0.6)
@@
 	)
 	(via
+		(at 78 66)
+		(size 0.6)
+		(drill 0.3)
+		(layers "F.Cu" "B.Cu")
+		(free yes)
+		(net 2)
+	)
+	(via
+		(at 127 77)
+		(size 0.6)
+		(drill 0.3)
+		(layers "F.Cu" "B.Cu")
+		(free yes)
+		(net 2)
+	)
+	(via
 		(at 121.5 100.5)
 		(size 0.6)
@@
 	)
 	(via
+		(at 87 89)
+		(size 0.6)
+		(drill 0.3)
+		(layers "F.Cu" "B.Cu")
+		(free yes)
+		(net 2)
+	)
+	(via
 		(at 116.5 77.5)
 		(size 0.6)
@@
 	)
 	(via
+		(at 122 83)
+		(size 0.6)
+		(drill 0.3)
+		(layers "F.Cu" "B.Cu")
+		(free yes)
+		(net 2)
+	)
+	(via
 		(at 108.75 107.25)
 		(size 0.6)
@@
 	)
 	(via
+		(at 43 110)
+		(size 0.6)
+		(drill 0.3)
+		(layers "F.Cu" "B.Cu")
+		(free yes)
+		(net 2)
+	)
+	(via
 		(at 121 54.75)
 		(size 0.6)
@@
 	)
 	(via
+		(at 128 49)
+		(size 0.6)
+		(drill 0.3)
+		(layers "F.Cu" "B.Cu")
+		(free yes)
+		(net 2)
+	)
+	(via
 		(at 132 59)
 		(size 0.6)
@@
 	)
 	(via
+		(at 68 66)
+		(size 0.6)
+		(drill 0.3)
+		(layers "F.Cu" "B.Cu")
+		(free yes)
+		(net 2)
+	)
+	(via
 		(at 82.3 128.236)
 		(size 0.6)
@@
 	)
 	(via
+		(at 89 124)
+		(size 0.6)
+		(drill 0.3)
+		(layers "F.Cu" "B.Cu")
+		(free yes)
+		(net 2)
+	)
+	(via
 		(at 121.5 106.75)
 		(size 0.6)
@@
 	)
 	(via
+		(at 63 78)
+		(size 0.6)
+		(drill 0.3)
+		(layers "F.Cu" "B.Cu")
+		(net 2)
+	)
+	(via
+		(at 117 65)
+		(size 0.6)
+		(drill 0.3)
+		(layers "F.Cu" "B.Cu")
+		(free yes)
+		(net 2)
+	)
+	(via
 		(at 109.00065 80.99935)
 		(size 0.6)
@@
 	)
 	(via
+		(at 111 57)
+		(size 0.6)
+		(drill 0.3)
+		(layers "F.Cu" "B.Cu")
+		(free yes)
+		(net 2)
+	)
+	(via
+		(at 116 22)
+		(size 0.6)
+		(drill 0.3)
+		(layers "F.Cu" "B.Cu")
+		(free yes)
+		(net 2)
+	)
+	(via
 		(at 80 73)
 		(size 0.6)
@@
 	)
 	(zone
+		(net 2)
+		(net_name "GND")
+		(layer "F.Cu")
+		(hatch edge 0.5)
+		(priority 3)
+		(connect_pads
+			(clearance 0.5)
+		)
+		(min_thickness 0.25)
+		(filled_areas_thickness no)
+		(fill yes
+			(thermal_gap 0.5)
+			(thermal_bridge_width 0.5)
+		)
+		(polygon
+			(pts
+				(xy 39 18) (xy 39 148) (xy 139 148) (xy 139 18)
+			)
+		)
+	)
+	(zone
