File: hw/if-2/connectors.kicad_sch (KiCad schematic)
At the start: 3 parts, among them J1 DB25_Socket, J2 PJ-102AH, J3 Conn_02x12_Top_Bottom

Commit message: Adding changes suggested by Dan
Connections:
- net R0_CTCSS_B: no longer J3.17 (Pin_17)
- new net R1_CTCSS_B: J3.17 (Pin_17)
Changed lines of the file:
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@@
 		)
 	)
-	(global_label "R0_CTCSS_B"
+	(global_label "R1_CTCSS_B"
 		(shape input)
 		(at 226.06 62.23 0)

Commit message: Ready to do layout on IF2 board
Parts:
- removed J3: Conn_02x12_Top_Bottom, symbol Connector_Generic:Conn_02x12_Top_Bottom
- added J3: Conn_02x12_Odd_Even, Connector_PinHeader_2.54mm:PinHeader_2x12_P2.54mm_Vertical, symbol Connector_Generic:Conn_02x12_Odd_Even
- J1: footprint (none) -> bruce-footprints:AMPHENOL_L77SDB25SA4CH4F
Connections:
- net +12V: now also J3.18 (Pin_18)
- net +3.3V: now also J3.22 (Pin_22)
- net +5V: now also J3.20 (Pin_20)
- net ADC_BCK: now also J3.5 (Pin_5)
- net ADC_DOUT: now also J3.7 (Pin_7)
- net ADC_LRCK: now also J3.3 (Pin_3)
- net ADC_SCK: now also J3.1 (Pin_1)
- net DAC_BCK: now also J3.13 (Pin_13)
- net DAC_DIN: now also J3.15 (Pin_15)
- net DAC_LRCK: now also J3.11 (Pin_11)
- net DAC_SCK: now also J3.9 (Pin_9)
- net GND: now also J3.23 (Pin_23), J3.24 (Pin_24)
- net R0_COS_B: now also J3.4 (Pin_4)
- net R0_CTCSS_B: now also J3.8 (Pin_8)
- net R0_PTT_B: now also J3.12 (Pin_12)
- net R1_COS_B: now also J3.6 (Pin_6)
- net R1_CTCSS_B: now also J3.10 (Pin_10)
- net R1_PTT_B: now also J3.14 (Pin_14)
- net ~{ADC_RST}: now also J3.2 (Pin_2)
Other:
- title: Connectors -> COS/CTCSS/PTT Controls (Radio 1)
Changed lines of the file:
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@@
 	(paper "USLetter")
 	(title_block
-		(title "Connectors")
+		(title "COS/CTCSS/PTT Controls (Radio 1)")
 		(date "2025-03-18")
 		(rev "2")
@@
 	)
 	(symbol
+		(lib_id "Connector_Generic:Conn_02x12_Odd_Even")
+		(at 205.74 64.77 0)
+		(unit 1)
+		(exclude_from_sim no)
+		(in_bom yes)
+		(on_board yes)
+		(dnp no)
+		(fields_autoplaced yes)
+		(property "Reference" "J3"
+			(at 207.01 45.72 0)
+			(effects
+				(font
+					(size 1.27 1.27)
+				)
+			)
+		)
+		(property "Value" "Conn_02x12_Odd_Even"
+			(at 207.01 48.26 0)
+			(effects
+				(font
+					(size 1.27 1.27)
+				)
+			)
+		)
+		(property "Footprint" "Connector_PinHeader_2.54mm:PinHeader_2x12_P2.54mm_Vertical"
+			(at 205.74 64.77 0)
+			(effects
+				(font
+					(size 1.27 1.27)
+				)
+				(hide yes)
+			)
+		)
+		(property "Datasheet" "~"
+			(at 205.74 64.77 0)
+			(effects
+				(font
+					(size 1.27 1.27)
+				)
+				(hide yes)
+			)
+		)
+		(property "Description" "Generic connector, double row, 02x12, odd/even pin numbering scheme (row 1 odd numbers, row 2 even numbers), script generated (kicad-library-utils/schlib/autogen/connector/)"
+			(at 205.74 64.77 0)
+			(effects
+				(font
+					(size 1.27 1.27)
+				)
+				(hide yes)
+			)
+		)
+		(pin "19"
+		)
+		(pin "13"
+		)
+		(pin "4"
+		)
+		(pin "8"
+		)
+		(pin "11"
+		)
+		(pin "3"
+		)
+		(pin "15"
+		)
+		(pin "9"
+		)
+		(pin "1"
+		)
+		(pin "17"
+		)
+		(pin "5"
+		)
+		(pin "7"
+		)
+		(pin "21"
+		)
+		(pin "23"
+		)
+		(pin "2"
+		)
+		(pin "6"
+		)
+		(pin "20"
+		)
+		(pin "10"
+		)
+		(pin "18"
+		)
+		(pin "16"
+		)
+		(pin "24"
+		)
+		(pin "22"
+		)
+		(pin "12"
+		)
+		(pin "14"
+		)
+		(instances
+			(project ""
+				(path "/a8c2d6aa-29bb-49bd-a367-0d62a0a32480/d264813b-cbb1-4d95-8ad4-d43dc0883cab"
+					(reference "J3")
+					(unit 1)
+				)
+			)
+		)
+	)
+	(symbol
 		(lib_id "power:GND")
 		(at 102.87 102.87 0)
@@
 				(path "/a8c2d6aa-29bb-49bd-a367-0d62a0a32480/d264813b-cbb1-4d95-8ad4-d43dc0883cab"
 					(reference "#PWR03")
-					(unit 1)
-				)
-			)
-		)
-	)
-	(symbol
-		(lib_id "Connector_Generic:Conn_02x12_Top_Bottom")
-		(at 205.74 64.77 0)
-		(unit 1)
-		(exclude_from_sim no)
-		(in_bom yes)
-		(on_board yes)
-		(dnp no)
-		(fields_autoplaced yes)
-		(property "Reference" "J3"
-			(at 207.01 45.72 0)
-			(effects
-				(font
-					(size 1.27 1.27)
-				)
-			)
-		)
-		(property "Value" "Conn_02x12_Top_Bottom"
-			(at 207.01 48.26 0)
-			(effects
-				(font
-					(size 1.27 1.27)
-				)
-			)
-		)
-		(property "Footprint" ""
-			(at 205.74 64.77 0)
-			(effects
-				(font
-					(size 1.27 1.27)
-				)
-				(hide yes)
-			)
-		)
-		(property "Datasheet" "~"
-			(at 205.74 64.77 0)
-			(effects
-				(font
-					(size 1.27 1.27)
-				)
-				(hide yes)
-			)
-		)
-		(property "Description" "Generic connector, double row, 02x12, top/bottom pin numbering scheme (row 1: 1...pins_per_row, row2: pins_per_row+1 ... num_pins), script generated (kicad-library-utils/schlib/autogen/connector/)"
-			(at 205.74 64.77 0)
-			(effects
-				(font
-					(size 1.27 1.27)
-				)
-				(hide yes)
-			)
-		)
-		(pin "9"
-		)
-		(pin "4"
-		)
-		(pin "2"
-		)
-		(pin "3"
-		)
-		(pin "6"
-		)
-		(pin "7"
-		)
-		(pin "10"
-		)
-		(pin "5"
-		)
-		(pin "1"
-		)
-		(pin "8"
-		)
-		(pin "20"
-		)
-		(pin "14"
-		)
-		(pin "18"
-		)
-		(pin "22"
-		)
-		(pin "17"
-		)
-		(pin "11"
-		)
-		(pin "15"
-		)
-		(pin "12"
-		)
-		(pin "16"
-		)
-		(pin "24"
-		)
-		(pin "23"
-		)
-		(pin "19"
-		)
-		(pin "21"
-		)
-		(pin "13"
-		)
-		(instances
-			(project "if-2"
-				(path "/a8c2d6aa-29bb-49bd-a367-0d62a0a32480/d264813b-cbb1-4d95-8ad4-d43dc0883cab"
-					(reference "J3")
 					(unit 1)
 				)
@@
 			)
 		)
-		(property "Footprint" ""
+		(property "Footprint" "bruce-footprints:AMPHENOL_L77SDB25SA4CH4F"
 			(at 120.65 66.04 0)
 			(effects

Commit message: Making progress on layout
Connections:
- net DAC_DIN: now also J3.11 (Pin_11); no longer J3.15 (Pin_15)
- net DAC_LRCK: now also J3.9 (Pin_9); no longer J3.11 (Pin_11)
- net DAC_SCK: now also J3.15 (Pin_15); no longer J3.9 (Pin_9)
Changed lines of the file:
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@@
 	(global_label "DAC_DIN"
 		(shape input)
+		(at 176.53 64.77 180)
+		(fields_autoplaced yes)
+		(effects
+			(font
+				(size 1.27 1.27)
+			)
+			(justify right)
+		)
+		(property "Intersheetrefs" "${INTERSHEET_REFS}"
+			(at 165.7433 64.77 0)
+			(effects
+				(font
+					(size 1.27 1.27)
+				)
+				(justify right)
+				(hide yes)
+			)
+		)
+	)
+	(global_label "R1_CTCSS_B"
+		(shape input)
+		(at 226.06 62.23 0)
+		(fields_autoplaced yes)
+		(effects
+			(font
+				(size 1.27 1.27)
+			)
+			(justify left)
+		)
+		(property "Intersheetrefs" "${INTERSHEET_REFS}"
+			(at 240.6565 62.23 0)
+			(effects
+				(font
+					(size 1.27 1.27)
+				)
+				(justify left)
+				(hide yes)
+			)
+		)
+	)
+	(global_label "DAC_SCK"
+		(shape input)
 		(at 176.53 69.85 180)
 		(fields_autoplaced yes)
@@
 		)
 		(property "Intersheetrefs" "${INTERSHEET_REFS}"
-			(at 165.7433 69.85 0)
-			(effects
-				(font
-					(size 1.27 1.27)
-				)
-				(justify right)
-				(hide yes)
-			)
-		)
-	)
-	(global_label "R1_CTCSS_B"
-		(shape input)
-		(at 226.06 62.23 0)
+			(at 165.1991 69.85 0)
+			(effects
+				(font
+					(size 1.27 1.27)
+				)
+				(justify right)
+				(hide yes)
+			)
+		)
+	)
+	(global_label "ADC_BCK"
+		(shape input)
+		(at 190.5 57.15 180)
+		(fields_autoplaced yes)
+		(effects
+			(font
+				(size 1.27 1.27)
+			)
+			(justify right)
+		)
+		(property "Intersheetrefs" "${INTERSHEET_REFS}"
+			(at 179.1086 57.15 0)
+			(effects
+				(font
+					(size 1.27 1.27)
+				)
+				(justify right)
+				(hide yes)
+			)
+		)
+	)
+	(global_label "R1_PTT"
+		(shape input)
+		(at 50.8 45.72 180)
+		(fields_autoplaced yes)
+		(effects
+			(font
+				(size 1.27 1.27)
+			)
+			(justify right)
+		)
+		(property "Intersheetrefs" "${INTERSHEET_REFS}"
+			(at 41.1625 45.72 0)
+			(effects
+				(font
+					(size 1.27 1.27)
+				)
+				(justify right)
+				(hide yes)
+			)
+		)
+	)
+	(global_label "12V_UNFUSED"
+		(shape input)
+		(at 93.98 147.32 0)
 		(fields_autoplaced yes)
 		(effects
@@
 		)
 		(property "Intersheetrefs" "${INTERSHEET_REFS}"
-			(at 240.6565 62.23 0)
+			(at 110.149 147.32 0)
 			(effects
 				(font
@@
 		)
 	)
-	(global_label "DAC_SCK"
+	(global_label "R0_COS"
+		(shape input)
+		(at 50.8 91.44 180)
+		(fields_autoplaced yes)
+		(effects
+			(font
+				(size 1.27 1.27)
+			)
+			(justify right)
+		)
+		(property "Intersheetrefs" "${INTERSHEET_REFS}"
+			(at 40.5577 91.44 0)
+			(effects
+				(font
+					(size 1.27 1.27)
+				)
+				(justify right)
+				(hide yes)
+			)
+		)
+	)
+	(global_label "ADC_SCK"
+		(shape input)
+		(at 190.5 52.07 180)
+		(fields_autoplaced yes)
+		(effects
+			(font
+				(size 1.27 1.27)
+			)
+			(justify right)
+		)
+		(property "Intersheetrefs" "${INTERSHEET_REFS}"
+			(at 179.1691 52.07 0)
+			(effects
+				(font
+					(size 1.27 1.27)
+				)
+				(justify right)
+				(hide yes)
+			)
+		)
+	)
+	(global_label "R0_CTCSS_B"
+		(shape input)
+		(at 243.84 59.69 0)
+		(fields_autoplaced yes)
+		(effects
+			(font
+				(size 1.27 1.27)
+			)
+			(justify left)
+		)
+		(property "Intersheetrefs" "${INTERSHEET_REFS}"
+			(at 258.4365 59.69 0)
+			(effects
+				(font
+					(size 1.27 1.27)
+				)
+				(justify left)
+				(hide yes)
+			)
+		)
+	)
+	(global_label "ADC_LRCK"
+		(shape input)
+		(at 175.26 54.61 180)
+		(fields_autoplaced yes)
+		(effects
+			(font
+				(size 1.27 1.27)
+			)
+			(justify right)
+		)
+		(property "Intersheetrefs" "${INTERSHEET_REFS}"
+			(at 162.8405 54.61 0)
+			(effects
+				(font
+					(size 1.27 1.27)
+				)
+				(justify right)
+				(hide yes)
+			)
+		)
+	)
+	(global_label "DAC_LRCK"
 		(shape input)
 		(at 190.5 62.23 180)
@@
 		)
 		(property "Intersheetrefs" "${INTERSHEET_REFS}"
-			(at 179.1691 62.23 0)
-			(effects
-				(font
-					(size 1.27 1.27)
-				)
-				(justify right)
-				(hide yes)
-			)
-		)
-	)
-	(global_label "ADC_BCK"
-		(shape input)
-		(at 190.5 57.15 180)
-		(fields_autoplaced yes)
-		(effects
-			(font
-				(size 1.27 1.27)
-			)
-			(justify right)
-		)
-		(property "Intersheetrefs" "${INTERSHEET_REFS}"
-			(at 179.1086 57.15 0)
-			(effects
-				(font
-					(size 1.27 1.27)
-				)
-				(justify right)
-				(hide yes)
-			)
-		)
-	)
-	(global_label "R1_PTT"
-		(shape input)
-		(at 50.8 45.72 180)
-		(fields_autoplaced yes)
-		(effects
-			(font
-				(size 1.27 1.27)
-			)
-			(justify right)
-		)
-		(property "Intersheetrefs" "${INTERSHEET_REFS}"
-			(at 41.1625 45.72 0)
-			(effects
-				(font
-					(size 1.27 1.27)
-				)
-				(justify right)
-				(hide yes)
-			)
-		)
-	)
-	(global_label "12V_UNFUSED"
-		(shape input)
-		(at 93.98 147.32 0)
-		(fields_autoplaced yes)
-		(effects
-			(font
-				(size 1.27 1.27)
-			)
-			(justify left)
-		)
-		(property "Intersheetrefs" "${INTERSHEET_REFS}"
-			(at 110.149 147.32 0)
-			(effects
-				(font
-					(size 1.27 1.27)
-				)
-				(justify left)
-				(hide yes)
-			)
-		)
-	)
-	(global_label "R0_COS"
-		(shape input)
-		(at 50.8 91.44 180)
-		(fields_autoplaced yes)
-		(effects
-			(font
-				(size 1.27 1.27)
-			)
-			(justify right)
-		)
-		(property "Intersheetrefs" "${INTERSHEET_REFS}"
-			(at 40.5577 91.44 0)
-			(effects
-				(font
-					(size 1.27 1.27)
-				)
-				(justify right)
-				(hide yes)
-			)
-		)
-	)
-	(global_label "ADC_SCK"
-		(shape input)
-		(at 190.5 52.07 180)
-		(fields_autoplaced yes)
-		(effects
-			(font
-				(size 1.27 1.27)
-			)
-			(justify right)
-		)
-		(property "Intersheetrefs" "${INTERSHEET_REFS}"
-			(at 179.1691 52.07 0)
-			(effects
-				(font
-					(size 1.27 1.27)
-				)
-				(justify right)
-				(hide yes)
-			)
-		)
-	)
-	(global_label "R0_CTCSS_B"
-		(shape input)
-		(at 243.84 59.69 0)
-		(fields_autoplaced yes)
-		(effects
-			(font
-				(size 1.27 1.27)
-			)
-			(justify left)
-		)
-		(property "Intersheetrefs" "${INTERSHEET_REFS}"
-			(at 258.4365 59.69 0)
-			(effects
-				(font
-					(size 1.27 1.27)
-				)
-				(justify left)
-				(hide yes)
-			)
-		)
-	)
-	(global_label "ADC_LRCK"
-		(shape input)
-		(at 175.26 54.61 180)
-		(fields_autoplaced yes)
-		(effects
-			(font
-				(size 1.27 1.27)
-			)
-			(justify right)
-		)
-		(property "Intersheetrefs" "${INTERSHEET_REFS}"
-			(at 162.8405 54.61 0)
-			(effects
-				(font
-					(size 1.27 1.27)
-				)
-				(justify right)
-				(hide yes)
-			)
-		)
-	)
-	(global_label "DAC_LRCK"
-		(shape input)
-		(at 176.53 64.77 180)
-		(fields_autoplaced yes)
-		(effects
-			(font
-				(size 1.27 1.27)
-			)
-			(justify right)
-		)
-		(property "Intersheetrefs" "${INTERSHEET_REFS}"
-			(at 164.1105 64.77 0)
-			(effects
-				(font
+			(at 178.0805 62.23 0)
+			(effects
+				(font

Commit message: Layout passes DRC!!
Connections:
- net R0_COS_B: now also J3.8 (Pin_8); no longer J3.4 (Pin_4)
- net R0_CTCSS_B: now also J3.6 (Pin_6); no longer J3.8 (Pin_8)
- net R0_PTT_B: now also J3.4 (Pin_4); no longer J3.12 (Pin_12)
- net R1_COS_B: now also J3.14 (Pin_14); no longer J3.6 (Pin_6)
- net R1_CTCSS_B: now also J3.12 (Pin_12); no longer J3.10 (Pin_10)
- net R1_PTT_B: now also J3.10 (Pin_10); no longer J3.14 (Pin_14)

Commit message: (Pre fab) Resolved warning with DB25 shell connections to ground
Parts:
- J1: symbol Connector:DB25_Socket -> symbol-library-1:DB25_Socket_With_Shell
Connections:
- net GND: now also J1.SH1 (Shell), J1.SH2 (Shell)
Changed lines of the file:
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@@
+	)
+	(junction
+		(at 138.43 67.31)
+		(diameter 0)
+		(color 0 0 0 0)
 	)
 	(junction
@@
 	(wire
 		(pts
+			(xy 138.43 62.23) (xy 138.43 67.31)
+		)
+		(stroke
+			(width 0)
+			(type default)
+		)
+	)
+	(wire
+		(pts
 			(xy 102.87 53.34) (xy 102.87 58.42)
 		)
@@
 		(pts
 			(xy 50.8 86.36) (xy 113.03 86.36)
+		)
+		(stroke
+			(width 0)
+			(type default)
+		)
+	)
+	(wire
+		(pts
+			(xy 132.08 62.23) (xy 138.43 62.23)
+		)
+		(stroke
+			(width 0)
+			(type default)
+		)
+	)
+	(wire
+		(pts
+			(xy 132.08 67.31) (xy 138.43 67.31)
 		)
 		(stroke
@@
 	)
 	(symbol
-		(lib_id "Connector:DB25_Socket")
+		(lib_id "symbol-library-1:DB25_Socket_With_Shell")
 		(at 120.65 66.04 0)
 		(mirror x)
@@
 		)
 		(pin "13"
+		)
+		(pin "SH2"
+		)
+		(pin "SH1"
 		)
 		(instances
@@
 					(unit 1)
 				)
+			)
+		)
+	)
+	(symbol
+		(lib_id "power:GND")
+		(at 138.43 67.31 0)
+		(unit 1)
+		(exclude_from_sim no)
+		(in_bom yes)
+		(on_board yes)
+		(dnp no)
+		(fields_autoplaced yes)
+		(property "Reference" "#PWR0156"
+			(at 138.43 73.66 0)
+			(effects
+				(font
+					(size 1.27 1.27)
+				)
+				(hide yes)
+			)
+		)
+		(property "Value" "GND"
+			(at 138.43 72.39 0)
+			(effects
+				(font
+					(size 1.27 1.27)
+				)
+			)
+		)
+		(property "Footprint" ""
+			(at 138.43 67.31 0)
+			(effects
+				(font
+					(size 1.27 1.27)
+				)
+				(hide yes)
+			)
+		)
+		(property "Datasheet" ""
+			(at 138.43 67.31 0)
+			(effects
+				(font
+					(size 1.27 1.27)
+				)
+				(hide yes)
+			)
+		)
+		(property "Description" "Power symbol creates a global label with name \"GND\" , ground"
+			(at 138.43 67.31 0)
+			(effects
+				(font
+					(size 1.27 1.27)
+				)
+				(hide yes)
+			)
+		)
+		(pin "1"
+		)
+		(instances
+			(project ""
+				(path "/a8c2d6aa-29bb-49bd-a367-0d62a0a32480/d264813b-cbb1-4d95-8ad4-d43dc0883cab"
+					(reference "#PWR0156")
+					(unit 1)
+				)
