File: hw/if-2/controls_0.kicad_sch (KiCad schematic)
At the start: 17 parts, among them Q1 MMBT3904, Q2 MMBT3904, U8 LTV-356T

Commit message: Documentation improvements, moved a OVP circuit
Connections:
- net R0_COS: now also D6.3 (COM)
- net R0_CTCSS: now also D7.3 (COM)
- net at Q1.1 (B), R23.1, R24.2: no longer D6.3 (COM)
- net at Q2.1 (B), R32.2, R33.1: no longer D7.3 (COM)
Other:
- note added: "Converts 5V logic to 3.3V logic. Works even if radio can't source +5 for a pull-up. IMPORTANT: Results in a logic inversion which will need to be undone in software."
- note added: "Protection from relay-induced (or other) transients. (SOT-323)"
- note added: "When Rx_CTCSS is +5V, base voltage is 1.6V."
- note removed: "Converts 5V logic to 3.3V logic. Works even if radio can't source +5 for a pull-up"
- note removed: "Protection from relay-induced (or other) transients."
- moved on the sheet: D6, D7
Changed lines of the file:
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@@
 	(title_block
 		(title "COS/CTCSS/PTT Controls (Radio 0)")
-		(date "2025-05-13")
+		(date "2025-05-31")
 		(rev "2")
 		(company "Bruce MacKinnon KC1FSZ")
@@
 	(text "Clamping OVP"
 		(exclude_from_sim no)
-		(at 114.3 83.82 0)
+		(at 82.296 82.55 0)
 		(effects
 			(font
@@
 	(text "Clamping OVP"
 		(exclude_from_sim no)
-		(at 113.03 22.86 0)
+		(at 83.82 21.082 0)
 		(effects
 			(font
@@
 		)
 	)
-	(text "Converts 5V logic to 3.3V logic. Works\neven if radio can't source +5 for a pull-up"
-		(exclude_from_sim no)
-		(at 118.11 128.27 0)
-		(effects
-			(font
-				(size 1.27 1.27)
-			)
-		)
-	)
-	(text "When Rx_COS is +5V, base \nvoltage is 1.6V."
+	(text "When Rx_CTCSS is +5V, base \nvoltage is 1.6V."
 		(exclude_from_sim no)
 		(at 151.13 123.19 0)
@@
 		)
 	)
-	(text "Converts 5V logic to 3.3V logic. Works\neven if radio can't source +5 for a pull-up"
+	(text "Converts 5V logic to 3.3V logic. Works\neven if radio can't source +5 for a pull-up.\nIMPORTANT: Results in a logic inversion which \nwill need to be undone in software."
 		(exclude_from_sim no)
 		(at 116.84 67.31 0)
@@
 		)
 	)
-	(text "Protection from relay-induced \n(or other) transients."
+	(text "Protection from relay-induced \n(or other) transients. (SOT-323)"
 		(exclude_from_sim no)
 		(at 98.552 165.1 0)
@@
 	)
 	(junction
-		(at 105.41 46.99)
+		(at 100.33 46.99)
 		(diameter 0)
 		(color 0 0 0 0)
 	)
 	(junction
-		(at 134.62 107.95)
+		(at 105.41 46.99)
 		(diameter 0)
 		(color 0 0 0 0)
@@
 	)
 	(junction
+		(at 101.6 107.95)
+		(diameter 0)
+		(color 0 0 0 0)
+	)
+	(junction
 		(at 144.78 40.64)
 		(diameter 0)
 		(color 0 0 0 0)
 	)
-	(junction
-		(at 133.35 46.99)
-		(diameter 0)
-		(color 0 0 0 0)
-	)
 	(wire
 		(pts
@@
 	(wire
 		(pts
-			(xy 133.35 29.21) (xy 133.35 46.99)
-		)
-		(stroke
-			(width 0)
-			(type default)
-		)
-	)
-	(wire
-		(pts
 			(xy 138.43 148.59) (xy 129.54 148.59)
 		)
@@
 	(wire
 		(pts
-			(xy 134.62 90.17) (xy 134.62 107.95)
+			(xy 97.79 26.67) (xy 100.33 26.67)
 		)
 		(stroke
@@
 	(wire
 		(pts
+			(xy 100.33 26.67) (xy 100.33 46.99)
+		)
+		(stroke
+			(width 0)
+			(type default)
+		)
+	)
+	(wire
+		(pts
 			(xy 144.78 101.6) (xy 144.78 102.87)
 		)
@@
 	(wire
 		(pts
-			(xy 130.81 107.95) (xy 134.62 107.95)
-		)
-		(stroke
-			(width 0)
-			(type default)
-		)
-	)
-	(wire
-		(pts
-			(xy 105.41 46.99) (xy 90.17 46.99)
+			(xy 130.81 107.95) (xy 137.16 107.95)
+		)
+		(stroke
+			(width 0)
+			(type default)
+		)
+	)
+	(wire
+		(pts
+			(xy 105.41 46.99) (xy 100.33 46.99)
 		)
 		(stroke
@@
 	(wire
 		(pts
-			(xy 129.54 29.21) (xy 133.35 29.21)
-		)
-		(stroke
-			(width 0)
-			(type default)
-		)
-	)
-	(wire
-		(pts
 			(xy 120.65 107.95) (xy 130.81 107.95)
 		)
@@
 	(wire
 		(pts
-			(xy 133.35 46.99) (xy 130.81 46.99)
-		)
-		(stroke
-			(width 0)
-			(type default)
-		)
-	)
-	(wire
-		(pts
 			(xy 105.41 107.95) (xy 105.41 109.22)
 		)
@@
 	(wire
 		(pts
-			(xy 129.54 90.17) (xy 134.62 90.17)
+			(xy 97.79 88.9) (xy 101.6 88.9)
 		)
 		(stroke
@@
 	(wire
 		(pts
+			(xy 100.33 46.99) (xy 90.17 46.99)
+		)
+		(stroke
+			(width 0)
+			(type default)
+		)
+	)
+	(wire
+		(pts
+			(xy 101.6 107.95) (xy 90.17 107.95)
+		)
+		(stroke
+			(width 0)
+			(type default)
+		)
+	)
+	(wire
+		(pts
 			(xy 130.81 46.99) (xy 130.81 49.53)
 		)
@@
 	(wire
 		(pts
-			(xy 105.41 107.95) (xy 90.17 107.95)
+			(xy 105.41 107.95) (xy 101.6 107.95)
 		)
 		(stroke
@@
 	(wire
 		(pts
-			(xy 134.62 107.95) (xy 137.16 107.95)
+			(xy 101.6 88.9) (xy 101.6 107.95)
 		)
 		(stroke
@@
 	(wire
 		(pts
-			(xy 137.16 46.99) (xy 133.35 46.99)
+			(xy 130.81 46.99) (xy 137.16 46.99)
 		)
 		(stroke
@@
 	(symbol
 		(lib_id "Diode:BAT54S")
-		(at 124.46 29.21 90)
+		(at 92.71 26.67 90)
 		(unit 1)
 		(exclude_from_sim no)
@@
 		(fields_autoplaced yes)
 		(property "Reference" "D6"
-			(at 121.92 27.9399 90)
+			(at 90.17 25.3999 90)
 			(effects
 				(font
@@
 		)
 		(property "Value" "BAT54S"
-			(at 121.92 30.4799 90)
+			(at 90.17 27.9399 90)
 			(effects
 				(font
@@
 		)
 		(property "Footprint" "Package_TO_SOT_SMD:SOT-23"
-			(at 121.285 27.305 0)
+			(at 89.535 24.765 0)
 			(effects
 				(font
@@
 		)
 		(property "Datasheet" "https://www.diodes.com/assets/Datasheets/ds11005.pdf"
-			(at 124.46 32.258 0)
+			(at 92.71 29.718 0)
 			(effects
 				(font
@@
 		)
 		(property "Description" "Vr 30V, If 200mA, Dual schottky barrier diode, in series, SOT-323"
-			(at 124.46 29.21 0)
+			(at 92.71 26.67 0)
 			(effects
 				(font
@@
 	(symbol
 		(lib_id "Diode:BAT54S")
-		(at 124.46 90.17 90)
+		(at 92.71 88.9 90)
 		(unit 1)
 		(exclude_from_sim no)
@@
 		(fields_autoplaced yes)
 		(property "Reference" "D7"
-			(at 121.92 88.8999 90)
+			(at 90.17 87.6299 90)
 			(effects
 				(font
@@
 		)
 		(property "Value" "BAT54S"
-			(at 121.92 91.4399 90)
+			(at 90.17 90.1699 90)
 			(effects
 				(font
@@
 		)
 		(property "Footprint" "Package_TO_SOT_SMD:SOT-23"
-			(at 121.285 88.265 0)
+			(at 89.535 86.995 0)
 			(effects
 				(font
@@
 		)
 		(property "Datasheet" "https://www.diodes.com/assets/Datasheets/ds11005.pdf"
-			(at 124.46 93.218 0)
+			(at 92.71 91.948 0)
 			(effects
 				(font
@@
 		)
 		(property "Description" "Vr 30V, If 200mA, Dual schottky barrier diode, in series, SOT-323"
-			(at 124.46 90.17 0)
+			(at 92.71 88.9 0)
 			(effects
 				(font
@@
 	(symbol
 		(lib_id "power:+5V")
-		(at 124.46 21.59 0)
+		(at 92.71 19.05 0)
 		(unit 1)
 		(exclude_from_sim no)
@@
 		(fields_autoplaced yes)
 		(property "Reference" "#PWR0102"
-			(at 124.46 25.4 0)
+			(at 92.71 22.86 0)
 			(effects
 				(font
@@
 		)
 		(property "Value" "+5V"
-			(at 124.46 16.51 0)
+			(at 92.71 13.97 0)
 			(effects
 				(font
@@
 		)
 		(property "Footprint" ""
-			(at 124.46 21.59 0)
+			(at 92.71 19.05 0)
 			(effects
 				(font
@@
 		)
 		(property "Datasheet" ""
-			(at 124.46 21.59 0)
+			(at 92.71 19.05 0)
 			(effects
 				(font
@@
 		)
 		(property "Description" "Power symbol creates a global label with name \"+5V\""
-			(at 124.46 21.59 0)
+			(at 92.71 19.05 0)
 			(effects
 				(font
@@
 	(symbol
 		(lib_id "power:GND")
-		(at 124.46 36.83 0)
+		(at 92.71 34.29 0)
 		(unit 1)
 		(exclude_from_sim no)
@@
 		(fields_autoplaced yes)
 		(property "Reference" "#PWR0103"
-			(at 124.46 43.18 0)
+			(at 92.71 40.64 0)
 			(effects
 				(font
@@
 		)
 		(property "Value" "GND"
-			(at 124.46 41.91 0)
+			(at 92.71 39.37 0)
 			(effects
 				(font
@@
 		)
 		(property "Footprint" ""
-			(at 124.46 36.83 0)
+			(at 92.71 34.29 0)
 			(effects
 				(font
@@
 		)
 		(property "Datasheet" ""
-			(at 124.46 36.83 0)
+			(at 92.71 34.29 0)
 			(effects
 				(font
@@
 		)
 		(property "Description" "Power symbol creates a global label with name \"GND\" , ground"
-			(at 124.46 36.83 0)
+			(at 92.71 34.29 0)
 			(effects
 				(font
@@
 	(symbol
 		(lib_id "power:+5V")
-		(at 124.46 82.55 0)
+		(at 92.71 81.28 0)
 		(unit 1)
 		(exclude_from_sim no)
@@
 		(fields_autoplaced yes)
 		(property "Reference" "#PWR0104"
-			(at 124.46 86.36 0)
+			(at 92.71 85.09 0)
 			(effects
 				(font
@@
 		)
 		(property "Value" "+5V"
-			(at 124.46 77.47 0)
+			(at 92.71 76.2 0)
 			(effects
 				(font
@@
 		)
 		(property "Footprint" ""
-			(at 124.46 82.55 0)
+			(at 92.71 81.28 0)
 			(effects
 				(font
@@
 		)
 		(property "Datasheet" ""
-			(at 124.46 82.55 0)
+			(at 92.71 81.28 0)
 			(effects
 				(font
@@
 		)
 		(property "Description" "Power symbol creates a global label with name \"+5V\""
-			(at 124.46 82.55 0)
+			(at 92.71 81.28 0)
 			(effects
 				(font
@@
 	(symbol
 		(lib_id "power:GND")
-		(at 124.46 97.79 0)
+		(at 92.71 96.52 0)
 		(unit 1)
 		(exclude_from_sim no)
@@
 		(fields_autoplaced yes)
 		(property "Reference" "#PWR0107"
-			(at 124.46 104.14 0)
+			(at 92.71 102.87 0)
 			(effects
 				(font
@@
 		)
 		(property "Value" "GND"
-			(at 124.46 102.87 0)
+			(at 92.71 101.6 0)
 			(effects
 				(font
@@
 		)
 		(property "Footprint" ""
-			(at 124.46 97.79 0)
+			(at 92.71 96.52 0)
 			(effects
 				(font
@@
 		)
 		(property "Datasheet" ""
-			(at 124.46 97.79 0)
+			(at 92.71 96.52 0)
 			(effects
 				(font
@@
 		)
 		(property "Description" "Power symbol creates a global label with name \"GND\" , ground"
-			(at 124.46 97.79 0)
-			(effects
-				(font
+			(at 92.71 96.52 0)
+			(effects
+				(font
