File: hw/if-2/audio_out_1.kicad_sch (KiCad schematic)
At the start: 18 parts, among them U91 TL072

Commit message: Updated audio file to 16K
Parts:
- R93: value 20k -> 4.7k
- R94: value 100k -> 4.7k
- U91: value TL072 -> TLV9152
Connections:
- net GND: now also RV91.1; no longer RV91.3
- net at C92.2: now also RV91.3; no longer RV91.1
Other:
- note added: "Audio output level trim. Adjust to reduce magnitude from DAC full-scale. CW increases gain."
- note removed: "Audio output level trim. Adjust to allow DAC full-scale."
- title: COS/CTCSS/PTT Controls (Radio 1) -> Audio Output (Radio 1)
Changed lines of the file:
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@@
 	(paper "USLetter")
 	(title_block
-		(title "COS/CTCSS/PTT Controls (Radio 1)")
+		(title "Audio Output (Radio 1)")
 		(date "2025-06-21")
 		(rev "3")
@@
 		)
 	)
-	(text "Audio output level trim.\nAdjust to allow DAC full-scale.\n"
-		(exclude_from_sim no)
-		(at 108.204 98.552 0)
+	(text "Audio output level trim.\nAdjust to reduce magnitude from DAC full-scale.\nCW increases gain.\n"
+		(exclude_from_sim no)
+		(at 108.712 98.806 0)
 		(effects
 			(font
@@
 			)
 		)
-		(property "Value" "TL072"
+		(property "Value" "TLV9152"
 			(at 217.17 46.9899 0)
 			(effects
@@
 			)
 		)
-		(property "Value" "TL072"
+		(property "Value" "TLV9152"
 			(at 85.09 69.85 0)
 			(effects
@@
 			)
 		)
-		(property "Value" "20k"
+		(property "Value" "4.7k"
 			(at 128.27 81.28 90)
 			(effects
@@
 		(lib_id "Device:R_Potentiometer_US")
 		(at 107.95 85.09 0)
-		(unit 1)
-		(exclude_from_sim no)
-		(in_bom yes)
-		(on_board yes)
-		(dnp no)
-		(fields_autoplaced yes)
+		(mirror x)
+		(unit 1)
+		(exclude_from_sim no)
+		(in_bom yes)
+		(on_board yes)
+		(dnp no)
 		(property "Reference" "RV91"
-			(at 105.41 83.8199 0)
+			(at 105.41 86.3601 0)
 			(effects
 				(font
@@
 		)
 		(property "Value" "50k"
-			(at 105.41 86.3599 0)
+			(at 105.41 83.8201 0)
 			(effects
 				(font
@@
 			)
 		)
-		(property "Value" "TL072"
+		(property "Value" "TLV9152"
 			(at 143.51 80.01 0)
 			(effects
@@
 			)
 		)
-		(property "Value" "100k"
+		(property "Value" "4.7k"
 			(at 143.51 67.31 90)
 			(effects
