File: hw/if-2/controls_1.kicad_sch (KiCad schematic)
At the start: 17 parts, among them Q11 MMBT3904, Q12 MMBT3904, Q14 2N7002

Commit message: Updating schematics, create new mini-board for radio interface
Parts:
- added R35, R36: 100, Resistor_SMD:R_0805_2012Metric_Pad1.20x1.40mm_HandSolder, symbol Device:R_Small_US
Connections:
- net R1_COS: now also R35.1; no longer C22.1, D12.3 (COM), R18.1, R20.2
- net R1_CTCSS: now also R36.1; no longer C20.1, D11.3 (COM), R17.1, R19.2
- new net: C22.1, D12.3 (COM), R18.1, R20.2, R35.2
- new net: C20.1, D11.3 (COM), R17.1, R19.2, R36.2
Other:
- note removed: "When Rx_COS is +5V, base voltage is 1.6V."
- note removed: "When Rx_CTCSS is +5V, base voltage is 1.6V."
Changed lines of the file:
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@@
 	(title_block
 		(title "COS/CTCSS/PTT Controls (Radio 1)")
-		(date "2025-06-21")
+		(date "2025-06-25")
 		(rev "3")
 		(company "Bruce MacKinnon KC1FSZ")
 		(comment 1 "Copyright (C) Bruce MacKinnon, 2025")
 		(comment 2 "NOT FOR COMMERCIAL USE")
-	)
-	(text "When Rx_COS is +5V, base \nvoltage is 1.6V."
-		(exclude_from_sim no)
-		(at 154.94 64.77 0)
-		(effects
-			(font
-				(size 1.27 1.27)
-			)
-		)
 	)
 	(text "Clamping OVP"
@@
 		)
 	)
-	(text "When Rx_CTCSS is +5V, base \nvoltage is 1.6V."
-		(exclude_from_sim no)
-		(at 154.94 125.73 0)
-		(effects
-			(font
-				(size 1.27 1.27)
-			)
-		)
-	)
 	(text "Radio Side"
 		(exclude_from_sim no)
-		(at 65.024 103.632 90)
+		(at 45.466 90.932 90)
 		(effects
 			(font
@@
 	(wire
 		(pts
+			(xy 74.93 49.53) (xy 82.55 49.53)
+		)
+		(stroke
+			(width 0)
+			(type default)
+		)
+	)
+	(wire
+		(pts
 			(xy 148.59 104.14) (xy 148.59 105.41)
 		)
@@
 	(wire
 		(pts
+			(xy 74.93 110.49) (xy 82.55 110.49)
+		)
+		(stroke
+			(width 0)
+			(type default)
+		)
+	)
+	(wire
+		(pts
 			(xy 96.52 146.05) (xy 125.73 146.05)
 		)
@@
 	(wire
 		(pts
-			(xy 104.14 110.49) (xy 93.98 110.49)
-		)
-		(stroke
-			(width 0)
-			(type default)
-		)
-	)
-	(wire
-		(pts
 			(xy 96.52 146.05) (xy 86.36 146.05)
 		)
@@
 	(wire
 		(pts
+			(xy 87.63 110.49) (xy 104.14 110.49)
+		)
+		(stroke
+			(width 0)
+			(type default)
+		)
+	)
+	(wire
+		(pts
 			(xy 162.56 151.13) (xy 149.86 151.13)
 		)
@@
 	(wire
 		(pts
+			(xy 87.63 49.53) (xy 102.87 49.53)
+		)
+		(stroke
+			(width 0)
+			(type default)
+		)
+	)
+	(wire
+		(pts
 			(xy 124.46 49.53) (xy 134.62 49.53)
 		)
@@
 		(pts
 			(xy 134.62 110.49) (xy 134.62 113.03)
-		)
-		(stroke
-			(width 0)
-			(type default)
-		)
-	)
-	(wire
-		(pts
-			(xy 102.87 49.53) (xy 93.98 49.53)
 		)
 		(stroke
@@
 	(global_label "R1_CTCSS"
 		(shape input)
-		(at 93.98 110.49 180)
+		(at 74.93 110.49 180)
 		(fields_autoplaced yes)
 		(effects
@@
 		)
 		(property "Intersheetrefs" "${INTERSHEET_REFS}"
-			(at 81.6211 110.49 0)
+			(at 62.5711 110.49 0)
 			(effects
 				(font
@@
 	(global_label "R1_COS"
 		(shape input)
-		(at 93.98 49.53 180)
+		(at 74.93 49.53 180)
 		(fields_autoplaced yes)
 		(effects
@@
 		)
 		(property "Intersheetrefs" "${INTERSHEET_REFS}"
-			(at 83.7377 49.53 0)
+			(at 64.6877 49.53 0)
 			(effects
 				(font
@@
 	)
 	(symbol
+		(lib_id "Device:R_Small_US")
+		(at 85.09 49.53 90)
+		(unit 1)
+		(exclude_from_sim no)
+		(in_bom yes)
+		(on_board yes)
+		(dnp no)
+		(fields_autoplaced yes)
+		(property "Reference" "R35"
+			(at 85.09 43.18 90)
+			(effects
+				(font
+					(size 1.27 1.27)
+				)
+			)
+		)
+		(property "Value" "100"
+			(at 85.09 45.72 90)
+			(effects
+				(font
+					(size 1.27 1.27)
+				)
+			)
+		)
+		(property "Footprint" "Resistor_SMD:R_0805_2012Metric_Pad1.20x1.40mm_HandSolder"
+			(at 85.09 49.53 0)
+			(effects
+				(font
+					(size 1.27 1.27)
+				)
+				(hide yes)
+			)
+		)
+		(property "Datasheet" "~"
+			(at 85.09 49.53 0)
+			(effects
+				(font
+					(size 1.27 1.27)
+				)
+				(hide yes)
+			)
+		)
+		(property "Description" "Resistor, small US symbol"
+			(at 85.09 49.53 0)
+			(effects
+				(font
+					(size 1.27 1.27)
+				)
+				(hide yes)
+			)
+		)
+		(pin "2"
+		)
+		(pin "1"
+		)
+		(instances
+			(project "if-2"
+				(path "/a8c2d6aa-29bb-49bd-a367-0d62a0a32480/aaca03b7-1394-4a9e-b9db-1ef93c5c7c02"
+					(reference "R35")
+					(unit 1)
+				)
+			)
+		)
+	)
+	(symbol
 		(lib_id "power:GND")
 		(at 148.59 54.61 0)
@@
 					(unit 1)
 				)
+			)
+		)
+	)
+	(symbol
+		(lib_id "Device:R_Small_US")
+		(at 85.09 110.49 90)
+		(unit 1)
+		(exclude_from_sim no)
+		(in_bom yes)
+		(on_board yes)
+		(dnp no)
+		(fields_autoplaced yes)
+		(property "Reference" "R36"
+			(at 85.09 104.14 90)
+			(effects
+				(font
+					(size 1.27 1.27)
+				)
+			)
+		)
+		(property "Value" "100"
+			(at 85.09 106.68 90)
+			(effects
+				(font
+					(size 1.27 1.27)
+				)
+			)
+		)
+		(property "Footprint" "Resistor_SMD:R_0805_2012Metric_Pad1.20x1.40mm_HandSolder"
+			(at 85.09 110.49 0)
+			(effects
+				(font
+					(size 1.27 1.27)
+				)
+				(hide yes)
+			)
+		)
+		(property "Datasheet" "~"
+			(at 85.09 110.49 0)
+			(effects
+				(font
+					(size 1.27 1.27)
+				)
+				(hide yes)
+			)
+		)
+		(property "Description" "Resistor, small US symbol"
+			(at 85.09 110.49 0)
+			(effects
+				(font
+					(size 1.27 1.27)
+				)
+				(hide yes)
+			)
+		)
+		(pin "2"
+		)
+		(pin "1"
+		)
+		(instances
+			(project "if-2"
+				(path "/a8c2d6aa-29bb-49bd-a367-0d62a0a32480/aaca03b7-1394-4a9e-b9db-1ef93c5c7c02"
+					(reference "R36")
+					(unit 1)
+				)
