File: hw/digital-2/connectors.kicad_sch (KiCad schematic)
At the start: 2 parts, among them J1 Debug, J3 RadioInterface

Commit message: Digital board complete
Parts:
- removed J1: Debug, symbol Connector_Generic:Conn_01x06
- added J1: Conn_01x07, Connector_PinHeader_2.54mm:PinHeader_1x07_P2.54mm_Vertical, symbol Connector_Generic:Conn_01x07
- added J2: LED0, Connector_PinHeader_2.54mm:PinHeader_1x02_P2.54mm_Vertical, symbol Connector_Generic:Conn_01x02
- added J4: I2C, Connector_PinHeader_2.54mm:PinHeader_1x03_P2.54mm_Vertical, symbol Connector_Generic:Conn_01x03
Connections:
- net +3.3V: now also J1.1 (Pin_1)
- net GND: now also J1.3 (Pin_3), J1.7 (Pin_7), J2.2 (Pin_2), J4.3 (Pin_3)
- net SWCLK: now also J1.2 (Pin_2)
- net SWDIO: now also J1.4 (Pin_4)
- net UART_RX: now also J1.6 (Pin_6)
- net UART_TX: now also J1.5 (Pin_5)
- new net I2C_SCL: J4.2 (Pin_2)
- new net I2C_SDA: J4.1 (Pin_1)
- new net LED0: J2.1 (Pin_1)

Commit message: All boards ready
Parts:
- removed J4: I2C, Connector_PinHeader_2.54mm:PinHeader_1x03_P2.54mm_Vertical, symbol Connector_Generic:Conn_01x03
- added J4: I2C, Connector_PinHeader_2.54mm:PinHeader_1x04_P2.54mm_Vertical, symbol Connector_Generic:Conn_01x04
Connections:
- net +3.3V: now also J1.7 (Pin_7), J4.3 (Pin_3); no longer J1.1 (Pin_1)
- net GND: now also J1.2 (Pin_2), J1.6 (Pin_6), J4.4 (Pin_4); no longer J1.3 (Pin_3), J1.7 (Pin_7)
- net I2C_SCL: now also J4.2 (Pin_2)
- net I2C_SDA: now also J4.1 (Pin_1)
- net SWCLK: now also J1.1 (Pin_1); no longer J1.2 (Pin_2)
- net SWDIO: now also J1.3 (Pin_3); no longer J1.4 (Pin_4)
- net UART_RX: now also J1.5 (Pin_5); no longer J1.6 (Pin_6)
- net UART_TX: now also J1.4 (Pin_4); no longer J1.5 (Pin_5)
Other:
- note added: "Debug/Power"
- note added: "I2C Accessory Connection"
- company: (none) -> Bruce MacKinnon KC1FSZ
- title: (none) -> Digital Repeater Controller
- moved on the sheet: J1
Changed lines of the file:
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@@
 	(generator "eeschema")
 	(generator_version "9.0")
-	(paper "A4")
+	(paper "USLetter")
+	(title_block
+		(title "Digital Repeater Controller")
+		(date "2025-05-13")
+		(rev "1")
+		(company "Bruce MacKinnon KC1FSZ")
+		(comment 1 "Copyright (C) 2025, Bruce MacKinnon")
+		(comment 2 "NOT FOR COMMERCIAL USE")
+	)
+	(text "I2C Accessory Connection"
+		(exclude_from_sim no)
+		(at 205.74 81.026 0)
+		(effects
+			(font
+				(size 1.27 1.27)
+			)
+		)
+	)
 	(text "Pin 15 is the DAC SCK"
 		(exclude_from_sim no)
@@
 			(font
 				(size 2.54 2.54)
+			)
+		)
+	)
+	(text "Debug/Power"
+		(exclude_from_sim no)
+		(at 84.074 150.368 0)
+		(effects
+			(font
+				(size 1.27 1.27)
 			)
 		)
@@
 	(wire
 		(pts
+			(xy 191.77 63.5) (xy 209.55 63.5)
+		)
+		(stroke
+			(width 0)
+			(type default)
+		)
+	)
+	(wire
+		(pts
 			(xy 140.97 132.08) (xy 140.97 128.27)
 		)
@@
 	(wire
 		(pts
+			(xy 205.74 66.04) (xy 209.55 66.04)
+		)
+		(stroke
+			(width 0)
+			(type default)
+		)
+	)
+	(wire
+		(pts
 			(xy 96.52 83.82) (xy 116.84 83.82)
 		)
@@
 	(wire
 		(pts
+			(xy 72.39 137.16) (xy 92.71 137.16)
+		)
+		(stroke
+			(width 0)
+			(type default)
+		)
+	)
+	(wire
+		(pts
 			(xy 193.04 58.42) (xy 209.55 58.42)
 		)
@@
 	(wire
 		(pts
-			(xy 209.55 63.5) (xy 205.74 63.5)
-		)
-		(stroke
-			(width 0)
-			(type default)
-		)
-	)
-	(wire
-		(pts
 			(xy 73.66 63.5) (xy 83.82 63.5)
 		)
@@
 	(wire
 		(pts
-			(xy 205.74 63.5) (xy 205.74 68.58)
+			(xy 205.74 66.04) (xy 205.74 71.12)
 		)
 		(stroke
@@
 	(symbol
 		(lib_id "Connector_Generic:Conn_01x07")
-		(at 97.79 127 0)
+		(at 97.79 129.54 0)
 		(unit 1)
 		(exclude_from_sim no)
@@
 		(fields_autoplaced yes)
 		(property "Reference" "J1"
-			(at 100.33 125.7299 0)
+			(at 100.33 128.2699 0)
 			(effects
 				(font
@@
 		)
 		(property "Value" "Conn_01x07"
-			(at 100.33 128.2699 0)
+			(at 100.33 130.8099 0)
 			(effects
 				(font
@@
 		)
 		(property "Footprint" "Connector_PinHeader_2.54mm:PinHeader_1x07_P2.54mm_Vertical"
-			(at 97.79 127 0)
+			(at 97.79 129.54 0)
 			(effects
 				(font
@@
 		)
 		(property "Datasheet" "~"
-			(at 97.79 127 0)
+			(at 97.79 129.54 0)
 			(effects
 				(font
@@
 		)
 		(property "Description" "Generic connector, single row, 01x07, script generated (kicad-library-utils/schlib/autogen/connector/)"
-			(at 97.79 127 0)
+			(at 97.79 129.54 0)
 			(effects
 				(font
@@
 	)
 	(symbol
-		(lib_id "power:+3.3V")
-		(at 92.71 119.38 0)
+		(lib_id "Connector_Generic:Conn_01x04")
+		(at 214.63 60.96 0)
 		(unit 1)
 		(exclude_from_sim no)
@@
 		(dnp no)
 		(fields_autoplaced yes)
+		(property "Reference" "J4"
+			(at 217.17 60.9599 0)
+			(effects
+				(font
+					(size 1.27 1.27)
+				)
+				(justify left)
+			)
+		)
+		(property "Value" "I2C"
+			(at 217.17 63.4999 0)
+			(effects
+				(font
+					(size 1.27 1.27)
+				)
+				(justify left)
+			)
+		)
+		(property "Footprint" "Connector_PinHeader_2.54mm:PinHeader_1x04_P2.54mm_Vertical"
+			(at 214.63 60.96 0)
+			(effects
+				(font
+					(size 1.27 1.27)
+				)
+				(hide yes)
+			)
+		)
+		(property "Datasheet" "~"
+			(at 214.63 60.96 0)
+			(effects
+				(font
+					(size 1.27 1.27)
+				)
+				(hide yes)
+			)
+		)
+		(property "Description" "Generic connector, single row, 01x04, script generated (kicad-library-utils/schlib/autogen/connector/)"
+			(at 214.63 60.96 0)
+			(effects
+				(font
+					(size 1.27 1.27)
+				)
+				(hide yes)
+			)
+		)
+		(pin "1"
+		)
+		(pin "4"
+		)
+		(pin "2"
+		)
+		(pin "3"
+		)
+		(instances
+			(project ""
+				(path "/ae78e9b9-9814-4a08-a50e-9313b5a684ff/50bc9b1a-b05e-4f42-89d2-9973ed2c2a8f"
+					(reference "J4")
+					(unit 1)
+				)
+			)
+		)
+	)
+	(symbol
+		(lib_id "power:+3.3V")
+		(at 72.39 137.16 90)
+		(unit 1)
+		(exclude_from_sim no)
+		(in_bom yes)
+		(on_board yes)
+		(dnp no)
+		(fields_autoplaced yes)
 		(property "Reference" "#PWR081"
-			(at 92.71 123.19 0)
+			(at 76.2 137.16 0)
 			(effects
 				(font
@@
 		)
 		(property "Value" "+3.3V"
-			(at 92.71 114.3 0)
-			(effects
-				(font
-					(size 1.27 1.27)
-				)
+			(at 68.58 137.1599 90)
+			(effects
+				(font
+					(size 1.27 1.27)
+				)
+				(justify left)
 			)
 		)
 		(property "Footprint" ""
-			(at 92.71 119.38 0)
+			(at 72.39 137.16 0)
 			(effects
 				(font
@@
 		)
 		(property "Datasheet" ""
-			(at 92.71 119.38 0)
+			(at 72.39 137.16 0)
 			(effects
 				(font
@@
 		)
 		(property "Description" "Power symbol creates a global label with name \"+3.3V\""
-			(at 92.71 119.38 0)
+			(at 72.39 137.16 0)
 			(effects
 				(font
@@
 	)
 	(symbol
-		(lib_id "Connector_Generic:Conn_01x03")
-		(at 214.63 60.96 0)
+		(lib_id "power:+3.3V")
+		(at 191.77 63.5 90)
 		(unit 1)
 		(exclude_from_sim no)
@@
 		(dnp no)
 		(fields_autoplaced yes)
-		(property "Reference" "J4"
-			(at 217.17 59.6899 0)
+		(property "Reference" "#PWR082"
+			(at 195.58 63.5 0)
+			(effects
+				(font
+					(size 1.27 1.27)
+				)
+				(hide yes)
+			)
+		)
+		(property "Value" "+3.3V"
+			(at 187.96 63.4999 90)
 			(effects
 				(font
@@
 			)
 		)
-		(property "Value" "I2C"
-			(at 217.17 62.2299 0)
-			(effects
-				(font
-					(size 1.27 1.27)
-				)
-				(justify left)
-			)
-		)
-		(property "Footprint" "Connector_PinHeader_2.54mm:PinHeader_1x03_P2.54mm_Vertical"
-			(at 214.63 60.96 0)
-			(effects
-				(font
-					(size 1.27 1.27)
-				)
-				(hide yes)
-			)
-		)
-		(property "Datasheet" "~"
-			(at 214.63 60.96 0)
-			(effects
-				(font
-					(size 1.27 1.27)
-				)
-				(hide yes)
-			)
-		)
-		(property "Description" "Generic connector, single row, 01x03, script generated (kicad-library-utils/schlib/autogen/connector/)"
-			(at 214.63 60.96 0)
+		(property "Footprint" ""
+			(at 191.77 63.5 0)
+			(effects
+				(font
+					(size 1.27 1.27)
+				)
+				(hide yes)
+			)
+		)
+		(property "Datasheet" ""
+			(at 191.77 63.5 0)
+			(effects
+				(font
+					(size 1.27 1.27)
+				)
+				(hide yes)
+			)
+		)
+		(property "Description" "Power symbol creates a global label with name \"+3.3V\""
+			(at 191.77 63.5 0)
 			(effects
 				(font
@@
 		(pin "1"
 		)
-		(pin "3"
-		)
-		(pin "2"
-		)
 		(instances
-			(project ""
+			(project "digital-2"
 				(path "/ae78e9b9-9814-4a08-a50e-9313b5a684ff/50bc9b1a-b05e-4f42-89d2-9973ed2c2a8f"
-					(reference "J4")
+					(reference "#PWR082")
 					(unit 1)
 				)
@@
 	(symbol
 		(lib_id "power:GND")
-		(at 205.74 68.58 0)
+		(at 205.74 71.12 0)
 		(unit 1)
 		(exclude_from_sim no)
@@
 		(fields_autoplaced yes)
 		(property "Reference" "#PWR04"
-			(at 205.74 74.93 0)
+			(at 205.74 77.47 0)
 			(effects
 				(font
@@
 		)
 		(property "Value" "GND"
-			(at 205.74 73.66 0)
+			(at 205.74 76.2 0)
 			(effects
 				(font
@@
 		)
 		(property "Footprint" ""
-			(at 205.74 68.58 0)
+			(at 205.74 71.12 0)
 			(effects
 				(font
@@
 		)
 		(property "Datasheet" ""
-			(at 205.74 68.58 0)
+			(at 205.74 71.12 0)
 			(effects
 				(font
@@
 		)
 		(property "Description" "Power symbol creates a global label with name \"GND\" , ground"
-			(at 205.74 68.58 0)
-			(effects
-				(font
+			(at 205.74 71.12 0)
+			(effects
+				(font
