File: hw/digital-2/controller.kicad_sch (KiCad schematic)
At the start: 1 part

Commit message: Digital board complete
Parts:
- added R1: 220, Resistor_SMD:R_0805_2012Metric_Pad1.20x1.40mm_HandSolder, symbol Device:R_US
Connections:
- net at A1.24 (GPIO18): now also R1.1
- net I2C_SDA: now reaches A1.4 (GPIO2)
- net I2C_SCL: now reaches A1.5 (GPIO3)
- new net LED0: R1.2
- no-connect marks 4 -> 13
Changed lines of the file:
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@@
 	(paper "A4")
 	(no_connect
+		(at 228.6 97.79)
+	)
+	(no_connect
+		(at 210.82 57.15)
+	)
+	(no_connect
+		(at 228.6 92.71)
+	)
+	(no_connect
 		(at 228.6 102.87)
 	)
 	(no_connect
+		(at 228.6 95.25)
+	)
+	(no_connect
 		(at 182.88 72.39)
 	)
 	(no_connect
+		(at 228.6 90.17)
+	)
+	(no_connect
+		(at 228.6 107.95)
+	)
+	(no_connect
+		(at 228.6 110.49)
+	)
+	(no_connect
 		(at 182.88 74.93)
 	)
@@
 		(at 228.6 118.11)
 	)
+	(no_connect
+		(at 205.74 57.15)
+	)
+	(no_connect
+		(at 228.6 113.03)
+	)
 	(wire
 		(pts
@@
 	(wire
 		(pts
+			(xy 228.6 87.63) (xy 255.27 87.63)
+		)
+		(stroke
+			(width 0)
+			(type default)
+		)
+	)
+	(wire
+		(pts
 			(xy 205.74 130.81) (xy 205.74 133.35)
 		)
@@
 	(wire
 		(pts
+			(xy 113.03 85.09) (xy 182.88 85.09)
+		)
+		(stroke
+			(width 0)
+			(type default)
+		)
+	)
+	(wire
+		(pts
+			(xy 125.73 87.63) (xy 182.88 87.63)
+		)
+		(stroke
+			(width 0)
+			(type default)
+		)
+	)
+	(wire
+		(pts
 			(xy 149.86 90.17) (xy 182.88 90.17)
 		)
@@
 	(wire
 		(pts
+			(xy 255.27 111.76) (xy 255.27 87.63)
+		)
+		(stroke
+			(width 0)
+			(type default)
+		)
+	)
+	(wire
+		(pts
 			(xy 161.29 64.77) (xy 182.88 64.77)
 		)
@@
 		)
 	)
+	(global_label "LED0"
+		(shape input)
+		(at 255.27 119.38 270)
+		(fields_autoplaced yes)
+		(effects
+			(font
+				(size 1.27 1.27)
+			)
+			(justify right)
+		)
+		(property "Intersheetrefs" "${INTERSHEET_REFS}"
+			(at 255.27 127.0218 90)
+			(effects
+				(font
+					(size 1.27 1.27)
+				)
+				(justify right)
+				(hide yes)
+			)
+		)
+	)
 	(global_label "DAC_BCK"
 		(shape input)
@@
 		)
 	)
+	(global_label "I2C_SCL"
+		(shape input)
+		(at 125.73 87.63 180)
+		(fields_autoplaced yes)
+		(effects
+			(font
+				(size 1.27 1.27)
+			)
+			(justify right)
+		)
+		(property "Intersheetrefs" "${INTERSHEET_REFS}"
+			(at 115.1853 87.63 0)
+			(effects
+				(font
+					(size 1.27 1.27)
+				)
+				(justify right)
+				(hide yes)
+			)
+		)
+	)
 	(global_label "R0_COS_B"
 		(shape input)
@@
 				)
 				(justify left)
+				(hide yes)
+			)
+		)
+	)
+	(global_label "I2C_SDA"
+		(shape input)
+		(at 113.03 85.09 180)
+		(fields_autoplaced yes)
+		(effects
+			(font
+				(size 1.27 1.27)
+			)
+			(justify right)
+		)
+		(property "Intersheetrefs" "${INTERSHEET_REFS}"
+			(at 102.4248 85.09 0)
+			(effects
+				(font
+					(size 1.27 1.27)
+				)
+				(justify right)
 				(hide yes)
 			)
@@
 					(unit 1)
 				)
+			)
+		)
+	)
+	(symbol
+		(lib_id "Device:R_US")
+		(at 255.27 115.57 0)
+		(unit 1)
+		(exclude_from_sim no)
+		(in_bom yes)
+		(on_board yes)
+		(dnp no)
+		(fields_autoplaced yes)
+		(property "Reference" "R1"
+			(at 261.62 115.57 90)
+			(effects
+				(font
+					(size 1.27 1.27)
+				)
+			)
+		)
+		(property "Value" "220"
+			(at 259.08 115.57 90)
+			(effects
+				(font
+					(size 1.27 1.27)
+				)
+			)
+		)
+		(property "Footprint" "Resistor_SMD:R_0805_2012Metric_Pad1.20x1.40mm_HandSolder"
+			(at 256.286 115.824 90)
+			(effects
+				(font
+					(size 1.27 1.27)
+				)
+				(hide yes)
+			)
+		)
+		(property "Datasheet" "~"
+			(at 255.27 115.57 0)
+			(effects
+				(font
+					(size 1.27 1.27)
+				)
+				(hide yes)
+			)
+		)
+		(property "Description" "Resistor, US symbol"
+			(at 255.27 115.57 0)
+			(effects
+				(font
+					(size 1.27 1.27)
+				)
+				(hide yes)
+			)
+		)
+		(pin "1"
+		)
+		(pin "2"
+		)
+		(instances
+			(project ""
+				(path "/ae78e9b9-9814-4a08-a50e-9313b5a684ff/fd063e56-decc-4d35-bde1-3529c411e91d"
+					(reference "R1")
+					(unit 1)
+				)

Commit message: All boards ready
Other:
- company: (none) -> Bruce MacKinnon KC1FSZ
- title: (none) -> Digital Repeater Controller
Changed lines of the file:
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@@
 	(generator "eeschema")
 	(generator_version "9.0")
-	(paper "A4")
+	(paper "USLetter")
+	(title_block
+		(title "Digital Repeater Controller")
+		(date "2025-05-13")
+		(rev "1")
+		(company "Bruce MacKinnon KC1FSZ")
+		(comment 1 "Copyright (C) 2025, Bruce MacKinnon")
+		(comment 2 "NOT FOR COMMERCIAL USE")
+	)
 	(no_connect
 		(at 228.6 97.79)
