File: hw/digital-2/digital-2.kicad_pcb (KiCad board)
At the start: 2 copper layers, 51 x 60 mm, 10 parts, among them J1 Conn_01x07, J2 LED0, J3 RadioInterface, J4 I2C

Commit message: All boards ready
Parts:
- J4: footprint Connector_PinHeader_2.54mm:PinHeader_1x03_P2.54mm_Vertical -> Connector_PinHeader_2.54mm:PinHeader_1x04_P2.54mm_Vertical
- moved J1 2.70 mm to (173.0, 124.5)
Connections:
- J1 pad 1: +3.3V -> SWCLK
- J1 pad 2: SWCLK -> GND
- J1 pad 3: GND -> SWDIO
- J1 pad 4: SWDIO -> UART_TX
- J1 pad 5: UART_TX -> UART_RX
- J1 pad 6: UART_RX -> GND
- J1 pad 7: GND -> +3.3V
- J4 pad 3: GND -> +3.3V
Routing:
- net +3.3V: track 106.8 -> 143.5 mm
- net I2C_SCL: track 9.37 -> 10.7 mm
- net I2C_SDA: track 10.4 -> 11.3 mm
Other:
- board text added: "2025-05 B KC1FSZ bruce@mackinnon.com"
- board text added: "33V"
- board text added: "Digital Repeater Controller"
- board text added: "SWD"
