File: hw/digital-2/digital-2.kicad_sch (KiCad schematic)
At the start: 0 parts

Commit message: Digital board complete
Parts:
- added H1, H2, H3, H4: MountingHole, MountingHole:MountingHole_3.5mm, symbol Mechanical:MountingHole

Commit message: All boards ready
Other:
- company: (none) -> Bruce MacKinnon KC1FSZ
- title: (none) -> Digital Repeater Controller
Changed lines of the file:
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@@
 	(generator "eeschema")
 	(generator_version "9.0")
-	(paper "A4")
+	(paper "USLetter")
+	(title_block
+		(title "Digital Repeater Controller")
+		(date "2025-05-13")
+		(rev "1")
+		(company "Bruce MacKinnon KC1FSZ")
+		(comment 1 "Copyright (C) 2025, Bruce MacKinnon")
+		(comment 2 "NOT FOR COMMERCIAL USE")
+	)
 	(symbol
 		(lib_id "Mechanical:MountingHole")
